File: tmc51x0-multiplexer-uart/microcontroller.kicad_sch (KiCad schematic)
At the start: 1 part

Commit message: Add components
Parts:
- added D401: D_SCHOTTKY_20V_1A, Janelia:DIOM3616X98N, symbol Janelia:D_SCHOTTKY_20V_1A
Connections:
- net ENABLE_TX_0: now reaches A401.1 (UART0-TX/I2C0-SDA/SPI0-RX/GP0)
- net ~{ENABLE_RX_2}: now reaches A401.10 (I2C1-SCL/SPI0-TX/GP7)
- net ENABLE_TX_3: now reaches A401.11 (UART1-TX/I2C0-SDA/SPI1-RX/GP8)
- net ~{ENABLE_RX_3}: now reaches A401.12 (UART1-RX/I2C0-SCL/SPI1-CS/GP9)
- net ENABLE_TX_4: now reaches A401.14 (I2C1-SDA/SPI1-SCK/GP10)
- net ~{ENABLE_RX_4}: now reaches A401.15 (I2C1-SCL/SPI1-TX/GP11)
- net ENABLE_TX_5: now reaches A401.16 (UART0-TX/I2C0-SDA/SPI1-RX/GP12)
- net ~{ENABLE_RX_5}: now reaches A401.17 (UART0-RX/I2C0-SCL/SPI1-CS/GP13)
- net ENABLE_TX_6: now reaches A401.19 (I2C1-SDA/SPI1-SCK/GP14)
- net ~{ENABLE_RX_0}: now reaches A401.2 (UART0-RX/I2C0-SCL/SPI0-CS/GP1)
- net ~{ENABLE_RX_6}: now reaches A401.20 (I2C1-SCL/SPI1-TX/GP15)
- net ENABLE_VCC: now reaches A401.29 (GP22)
- net ENABLE_TX_7: now reaches A401.31 (I2C1-SDA/ADC0/GP26)
- net ~{ENABLE_RX_7}: now reaches A401.32 (I2C1-SCL/ADC1/GP27)
- net +3.3V: now reaches A401.36 (3V3(OUT))
- net GND: now reaches A401.38 (GND)
- net VSYS: now reaches A401.39 (VSYS)
- net VSYS: now also D401.1 (K)
- net ENABLE_TX_1: now reaches A401.4 (I2C1-SDA/SPI0-SCK/GP2)
- net ~{ENABLE_RX_1}: now reaches A401.5 (I2C1-SCL/SPI0-TX/GP3)
- net TX: now reaches A401.6 (UART1-TX/I2C0-SDA/SPI0-RX/GP4)
- net RX: now reaches A401.7 (UART1-RX/I2C0-SCL/SPI0-CS/GP5)
- net ENABLE_TX_2: now reaches A401.9 (I2C1-SDA/SPI0-SCK/GP6)
- new net +5V: D401.2 (A)
- no-connect marks 0 -> 12
Changed lines of the file:
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@@
 (kicad_sch (version 20230121) (generator eeschema)
   (paper "A4")
+  (no_connect (at 180.34 81.28))
+  (no_connect (at 180.34 99.06))
+  (no_connect (at 93.98 86.36))
+  (no_connect (at 180.34 68.58))
+  (no_connect (at 180.34 86.36))
+  (no_connect (at 180.34 93.98))
+  (no_connect (at 180.34 111.76))
+  (no_connect (at 180.34 76.2))
+  (no_connect (at 93.98 99.06))
+  (no_connect (at 93.98 73.66))
+  (no_connect (at 93.98 111.76))
+  (no_connect (at 180.34 83.82))
+  (wire (pts (xy 91.44 109.22) (xy 93.98 109.22))
+    (stroke (width 0) (type default))
+  )
+  (wire (pts (xy 91.44 78.74) (xy 93.98 78.74))
+    (stroke (width 0) (type default))
+  )
+  (wire (pts (xy 91.44 68.58) (xy 93.98 68.58))
+    (stroke (width 0) (type default))
+  )
+  (wire (pts (xy 91.44 93.98) (xy 93.98 93.98))
+    (stroke (width 0) (type default))
+  )
+  (wire (pts (xy 91.44 71.12) (xy 93.98 71.12))
+    (stroke (width 0) (type default))
+  )
+  (wire (pts (xy 54.61 49.53) (xy 57.15 49.53))
+    (stroke (width 0) (type default))
+  )
+  (wire (pts (xy 91.44 106.68) (xy 93.98 106.68))
+    (stroke (width 0) (type default))
+  )
+  (wire (pts (xy 180.34 96.52) (xy 182.88 96.52))
+    (stroke (width 0) (type default))
+  )
+  (wire (pts (xy 91.44 76.2) (xy 93.98 76.2))
+    (stroke (width 0) (type default))
+  )
+  (wire (pts (xy 91.44 104.14) (xy 93.98 104.14))
+    (stroke (width 0) (type default))
+  )
+  (wire (pts (xy 180.34 78.74) (xy 182.88 78.74))
+    (stroke (width 0) (type default))
+  )
+  (wire (pts (xy 54.61 52.07) (xy 57.15 52.07))
+    (stroke (width 0) (type default))
+  )
+  (wire (pts (xy 91.44 83.82) (xy 93.98 83.82))
+    (stroke (width 0) (type default))
+  )
+  (wire (pts (xy 91.44 116.84) (xy 93.98 116.84))
+    (stroke (width 0) (type default))
+  )
+  (wire (pts (xy 182.88 91.44) (xy 180.34 91.44))
+    (stroke (width 0) (type default))
+  )
+  (wire (pts (xy 180.34 73.66) (xy 182.88 73.66))
+    (stroke (width 0) (type default))
+  )
+  (wire (pts (xy 182.88 88.9) (xy 180.34 88.9))
+    (stroke (width 0) (type default))
+  )
+  (wire (pts (xy 91.44 81.28) (xy 93.98 81.28))
+    (stroke (width 0) (type default))
+  )
+  (wire (pts (xy 91.44 88.9) (xy 93.98 88.9))
+    (stroke (width 0) (type default))
+  )
+  (wire (pts (xy 91.44 101.6) (xy 93.98 101.6))
+    (stroke (width 0) (type default))
+  )
+  (wire (pts (xy 140.97 58.42) (xy 143.51 58.42))
+    (stroke (width 0) (type default))
+  )
+  (wire (pts (xy 91.44 114.3) (xy 93.98 114.3))
+    (stroke (width 0) (type default))
+  )
+  (wire (pts (xy 91.44 96.52) (xy 93.98 96.52))
+    (stroke (width 0) (type default))
+  )
+  (wire (pts (xy 135.89 58.42) (xy 133.35 58.42))
+    (stroke (width 0) (type default))
+  )
+  (wire (pts (xy 54.61 46.99) (xy 57.15 46.99))
+    (stroke (width 0) (type default))
+  )
+  (wire (pts (xy 180.34 71.12) (xy 182.88 71.12))
+    (stroke (width 0) (type default))
+  )
+  (wire (pts (xy 91.44 91.44) (xy 93.98 91.44))
+    (stroke (width 0) (type default))
+  )
+  (label "+3.3V" (at 57.15 49.53 0) (fields_autoplaced)
+    (effects (font (size 1.27 1.27)) (justify left bottom))
+  )
+  (label "+3.3V" (at 182.88 78.74 0) (fields_autoplaced)
+    (effects (font (size 1.27 1.27)) (justify left bottom))
+  )
+  (label "+5V" (at 133.35 58.42 180) (fields_autoplaced)
+    (effects (font (size 1.27 1.27)) (justify right bottom))
+  )
+  (label "VSYS" (at 182.88 71.12 0) (fields_autoplaced)
+    (effects (font (size 1.27 1.27)) (justify left bottom))
+  )
+  (label "VSYS" (at 143.51 58.42 0) (fields_autoplaced)
+    (effects (font (size 1.27 1.27)) (justify left bottom))
+  )
+  (label "+5V" (at 57.15 46.99 0) (fields_autoplaced)
+    (effects (font (size 1.27 1.27)) (justify left bottom))
+  )
+  (label "GND" (at 57.15 52.07 0) (fields_autoplaced)
+    (effects (font (size 1.27 1.27)) (justify left bottom))
+  )
+  (label "GND" (at 182.88 73.66 0) (fields_autoplaced)
+    (effects (font (size 1.27 1.27)) (justify left bottom))
+  )
+  (hierarchical_label "ENABLE_VCC" (shape output) (at 182.88 96.52 0) (fields_autoplaced)
+    (effects (font (size 1.27 1.27)) (justify left))
+  )
+  (hierarchical_label "~{ENABLE_RX_0}" (shape output) (at 91.44 71.12 180) (fields_autoplaced)
+    (effects (font (size 1.27 1.27)) (justify right))
+  )
+  (hierarchical_label "~{ENABLE_RX_7}" (shape output) (at 182.88 88.9 0) (fields_autoplaced)
+    (effects (font (size 1.27 1.27)) (justify left))
+  )
+  (hierarchical_label "~{ENABLE_RX_6}" (shape output) (at 91.44 116.84 180) (fields_autoplaced)
+    (effects (font (size 1.27 1.27)) (justify right))
+  )
+  (hierarchical_label "ENABLE_TX_4" (shape output) (at 91.44 101.6 180) (fields_autoplaced)
+    (effects (font (size 1.27 1.27)) (justify right))
+  )
+  (hierarchical_label "+5V" (shape passive) (at 54.61 46.99 180) (fields_autoplaced)
+    (effects (font (size 1.27 1.27)) (justify right))
+  )
+  (hierarchical_label "TX" (shape output) (at 91.44 81.28 180) (fields_autoplaced)
+    (effects (font (size 1.27 1.27)) (justify right))
+  )
+  (hierarchical_label "ENABLE_TX_0" (shape output) (at 91.44 68.58 180) (fields_autoplaced)
+    (effects (font (size 1.27 1.27)) (justify right))
+  )
+  (hierarchical_label "~{ENABLE_RX_3}" (shape output) (at 91.44 96.52 180) (fields_autoplaced)
+    (effects (font (size 1.27 1.27)) (justify right))
+  )
+  (hierarchical_label "GND" (shape passive) (at 54.61 52.07 180) (fields_autoplaced)
+    (effects (font (size 1.27 1.27)) (justify right))
+  )
+  (hierarchical_label "ENABLE_TX_5" (shape output) (at 91.44 106.68 180) (fields_autoplaced)
+    (effects (font (size 1.27 1.27)) (justify right))
+  )
+  (hierarchical_label "ENABLE_TX_6" (shape output) (at 91.44 114.3 180) (fields_autoplaced)
+    (effects (font (size 1.27 1.27)) (justify right))
+  )
+  (hierarchical_label "ENABLE_TX_3" (shape output) (at 91.44 93.98 180) (fields_autoplaced)
+    (effects (font (size 1.27 1.27)) (justify right))
+  )
+  (hierarchical_label "ENABLE_TX_1" (shape output) (at 91.44 76.2 180) (fields_autoplaced)
+    (effects (font (size 1.27 1.27)) (justify right))
+  )
+  (hierarchical_label "~{ENABLE_RX_2}" (shape output) (at 91.44 91.44 180) (fields_autoplaced)
+    (effects (font (size 1.27 1.27)) (justify right))
+  )
+  (hierarchical_label "ENABLE_TX_2" (shape output) (at 91.44 88.9 180) (fields_autoplaced)
+    (effects (font (size 1.27 1.27)) (justify right))
+  )
+  (hierarchical_label "RX" (shape input) (at 91.44 83.82 180) (fields_autoplaced)
+    (effects (font (size 1.27 1.27)) (justify right))
+  )
+  (hierarchical_label "~{ENABLE_RX_5}" (shape output) (at 91.44 109.22 180) (fields_autoplaced)
+    (effects (font (size 1.27 1.27)) (justify right))
+  )
+  (hierarchical_label "ENABLE_TX_7" (shape output) (at 182.88 91.44 0) (fields_autoplaced)
+    (effects (font (size 1.27 1.27)) (justify left))
+  )
+  (hierarchical_label "+3.3V" (shape passive) (at 54.61 49.53 180) (fields_autoplaced)
+    (effects (font (size 1.27 1.27)) (justify right))
+  )
+  (hierarchical_label "~{ENABLE_RX_1}" (shape output) (at 91.44 78.74 180) (fields_autoplaced)
+    (effects (font (size 1.27 1.27)) (justify right))
+  )
+  (hierarchical_label "~{ENABLE_RX_4}" (shape output) (at 91.44 104.14 180) (fields_autoplaced)
+    (effects (font (size 1.27 1.27)) (justify right))
+  )
   (symbol (lib_id "Janelia:PICO-W5500-EVB_HEADER_HOLES") (at 137.16 92.71 0) (unit 1)
     (in_bom no) (on_board yes) (dnp no) (fields_autoplaced)
@@
         )
       )
+    )
+  )
+  (symbol (lib_id "Janelia:D_SCHOTTKY_20V_1A") (at 138.43 58.42 180) (unit 1)
+    (in_bom yes) (on_board yes) (dnp no) (fields_autoplaced)
+    (property "Reference" "D401" (at 138.557 54.61 0)
+      (effects (font (size 1.27 1.27)))
+    )
+    (property "Value" "D_SCHOTTKY_20V_1A" (at 145.542 56.388 0)
+      (effects (font (size 1.27 1.27)) (justify left) hide)
+    )
+    (property "Footprint" "Janelia:DIOM3616X98N" (at 142.24 57.912 0)
+      (effects (font (size 1.524 1.524)) hide)
+    )
+    (property "Datasheet" "" (at 139.7 60.452 0)
+      (effects (font (size 1.524 1.524)) hide)
+    )
+    (property "Vendor" "Digi-Key" (at 137.16 62.992 0)
+      (effects (font (size 1.524 1.524)) hide)
+    )
+    (property "Vendor Part Number" "MBR120VLSFT1GOSCT-ND" (at 134.62 65.532 0)
+      (effects (font (size 1.524 1.524)) hide)
+    )
+    (property "Synopsis" "DIODE SCHOTTKY 20V 1A" (at 132.08 68.072 0)
+      (effects (font (size 1.524 1.524)) hide)
+    )
+    (property "Manufacturer" "onsemi" (at 138.43 58.42 0)
+      (effects (font (size 1.27 1.27)) hide)
+    )
+    (property "Manufacturer Part Number" "MBR120VLSFT1G" (at 138.43 58.42 0)
+      (effects (font (size 1.27 1.27)) hide)
+    )
+    (property "Package" " SOD123FL" (at 138.43 58.42 0)
+      (effects (font (size 1.27 1.27)) hide)
+    )
+    (property "Sim.Enable" "0" (at 138.43 58.42 0)
+      (effects (font (size 1.27 1.27)) hide)
+    )
+    (property "LCSC" "C223608" (at 138.43 58.42 0)
+      (effects (font (size 1.27 1.27)) hide)
+    )
+    (pin "1")
+    (pin "2")
+    (instances
+      (project "tmc51x0-multiplexer-uart"
+        (path "/df2b2e89-e055-4140-95de-f1df723db034/90ad6836-1738-4b32-a341-0a0b169f4662"
+          (reference "D401") (unit 1)
+        )
+      )
