File: tmc51x0-multiplexer-uart/motor.kicad_sch (KiCad schematic)
At the start: 1 part, among them U501 MAX13431E

Commit message: Add components
Parts:
- added C501: 0.1uF_100V, Janelia:C_0402_1005Metric, symbol Janelia:C_0.1uF_100V_0402
- added C502: 1uF_35V, Janelia:C_0402_1005Metric, symbol Janelia:C_1uF_35V_0402
- added D501: D, Janelia:D_SMB, symbol Janelia:D_1.25V@2A_400V
- added D502: D_Zener_47V_1W, Janelia:D_SMA, symbol Janelia:D_Zener_47V_1W
- added J501: FFC_P1mm_BOT_RA_SMD, Janelia:CONN_C2914097, symbol Janelia:Conn_01x10_FFC_P1mm_BOT_RA_SMD
- added R501: 0.24, Janelia:R_2512_6332Metric, symbol Janelia:R_0.240_1W_2512
- added R502: 120, Janelia:R_0402_1005Metric, symbol Janelia:R_120_0402
Connections:
- net +3.3V: now reaches U501.1 (VL)
- net +3.3V: now also C501.1
- net RX: now reaches U501.2 (RO)
- net ENABLE_TX: now reaches U501.3 (DE)
- net ~{ENABLE_RX}: now reaches U501.4 (~{RE})
- net TX: now reaches U501.5 (DI)
- net GND: now reaches U501.6 (GND)
- net GND: now also U501.11 (EP), C501.2, C502.2, D502.2 (A), J501.5 (Pin_5), J501.6 (Pin_6), J501.7 (Pin_7), J501.8 (Pin_8)
- net SWP: now reaches U501.8 (A)
- net SWP: now also J501.9 (Pin_9), R502.1
- new net +5V: C502.1, U501.10 (VCC)
- new net SWN: J501.10 (Pin_10), R502.2, U501.9 (B)
- new net VAA: R501.1
- new net VBB: D501.2 (A), D502.1 (K), R501.2
- new net VCC: D501.1 (K), J501.1 (Pin_1), J501.2 (Pin_2), J501.3 (Pin_3), J501.4 (Pin_4)
