File: tmc51x0-multiplexer-uart/power.kicad_sch (KiCad schematic)
At the start: 18 parts, among them J301 Molex_Pico-SPOX_Horizontal, J302 Molex_Pico-Lock-PLUS_Vertical, M301 Fan_5VDC_25x25x8mm, Q301 MOSFET-N-CH, U301 Switching_5V_500mA, U302 Linear_3.3V_1A

Commit message: Add components
Parts:
- removed C301: 2.2uF_100V, Janelia:C_0805_2012Metric, symbol Janelia:C_2.2uF_100V_0805
- removed C302: 47uF_10V, Janelia:C_0805_2012Metric, symbol Janelia:C_47uF_10V_0805
- removed C303, C304, C305: 1uF_25V, Janelia:C_0402_1005Metric, symbol Janelia:C_1uF_25V_0402
- removed D301: LED_RED, Janelia:LED_0402-1005_KNB, symbol Janelia:LED_KNB_20mA_RED_1.95V_0402
- removed D302: LED_GRN, Janelia:LED_0402-1005_KNB, symbol Janelia:LED_KNB_20mA_GRN_2.1V_0402
- removed D303: LED_YEL, Janelia:LED_0402-1005_KNB, symbol Janelia:LED_KNB_20mA_YEL_2V_0402
- removed J301: Molex_Pico-SPOX_Horizontal, Janelia:Molex_Pico-SPOX-87438_1x02-P1.5mm_Horizontal, symbol Janelia:Conn_01x02_P1.5mm_Molex_Pico-SPOX-87438_Horizontal
- removed J302: Molex_Pico-Lock-PLUS_Vertical, Janelia:Molex_Micro-Lock-PLUS-505568_1x02_P1.25mm_Vertical, symbol Janelia:Conn_01x02_P1.25mm_Molex_Micro-Lock-PLUS-505568_Vertical
- removed L301: 150uH_553mA, Janelia:IND_CB_SD25, symbol Janelia:L_150uH_553mA
- removed M301: Fan_5VDC_25x25x8mm, Janelia:FAN_5VDC_25x25x8mm, symbol Janelia:Fan_5VDC_25x25x8mm
- removed Q301: MOSFET-N-CH, Janelia:XFDFN-3, symbol Janelia:MOSFET-N-CH-EN-CSD17483F4
- removed R301: 2.32k, Janelia:R_0805_2012Metric, symbol Janelia:R_2.32k_1W_0805
- removed R302: 64.9, Janelia:R_0402_1005Metric, symbol Janelia:R_64.9_0.1W_0402
- removed R303: 249, Janelia:R_0402_1005Metric, symbol Janelia:R_249_0.06W_0402
- removed U301: Switching_5V_500mA, Janelia:Texas_S-PVSON-N10_ThermalVias, symbol Janelia:Regulator_Switching_5V_500mA_LM5166X
- removed U302: Linear_3.3V_1A, Janelia:TPS737Q1, symbol Janelia:Regulator_Linear_3.3V_1A_5.5Vin_TPS73733QDRBRQ1
- added D301: D_50V_15A, Janelia:POWERDI5_DIO, symbol Janelia:D_50V_15A
- added Q301: MOSFET-P-CH-EN_60V_50A, Janelia:TO-252-2, symbol Janelia:MOSFET-P-CH-EN_60V_50A
- added Q302: MOSFET-N-CH-EN_100V_260mA, Janelia:SOT-23, symbol Janelia:MOSFET-N-CH-EN_100V_260mA
- added T301: TERM_BLK_HDR_2POS_90DEG_0.2IN, Janelia:PHOENIX_1757242, symbol Janelia:TERM_BLK_HDR_2POS_90DEG_0.2IN
Connections:
- net GND: now also Q302.2 (S), T301.2 (P2)
- new net ENABLE_VCC: Q302.1 (G)
- new net VAA: D301.2 (A), T301.1 (P1)
- new net VBB: D301.1 (K), Q301.3 (S)
- no-connect marks 4 -> 0

Commit message: Add components
Parts:
- added R301: 1k, Janelia:R_0402_1005Metric, symbol Janelia:R_1k_0402
- added R302: 3.6k, Janelia:R_0402_1005Metric, symbol Janelia:R_3.6k_0402
Connections:
- net VBB: now also R301.1
- net VCC: now also Q301.2 (D)
- net ~{ENABLE_VCC}: now reaches Q301.1 (G)
- net ~{ENABLE_VCC}: now also R301.2, R302.1
- net at Q302.3 (D): now also R302.2
Other:
- moved on the sheet: Q301, Q302
