File: tmc5130-uart-multiplexer/tmc5130-uart-multiplexer.kicad_pcb (KiCad board)
At the start: 4 copper layers, 40 x 40 mm, 103 parts, among them J1301 Connector_USB_C_Receptacle, J301 Molex_Pico-SPOX_Horizontal, J302 Molex_Pico-Lock-PLUS_Vertical, J401 Molex_Pico-SPOX_Horizontal, J402 Molex_Pico-Clasp_Horizontal, M301 Fan_5VDC_25x25x8mm, Q301 MOSFET-N-CH, SW1301 Switch_Tactile_SPST-NO_SMT_Si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, U1001 BUK7D36-60EX, U1101 BUK7D36-60EX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

Commit message: tmc51x0-multiplexer-uart -> tmc5130-uart-multiplexer
Other:
- board text added: "https://github.com/janelia-kicad/tmc5130-uart-multiplexer"
- board text added: "tmc5130-uart-multiplexer v1.0 2024/05 48V 1.6A RMS 2.2A PEAK"
- board text removed: "https://github.com/janelia-kicad/tmc51x0-multiplexer-uart"
- board text removed: "tmc51x0-multiplexer-uart v1.0 2024/05 48V 1.6A RMS 2.2A PEAK"
Changed lines of the file:
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@@
   (paper "A4")
   (title_block
-    (title "tmc51x0-multiplexer-uart")
+    (title "tmc5130-uart-multiplexer")
     (date "2024-05-08")
     (rev "1.0")
@@
     (effects (font (size 1 0.6) (thickness 0.15) bold))
   )
-  (gr_text "tmc51x0-multiplexer-uart\nv1.0 2024/05\n48V 1.6A RMS 2.2A PEAK" (at 158.4 116.1) (layer "F.SilkS")
+  (gr_text "tmc5130-uart-multiplexer\nv1.0 2024/05\n48V 1.6A RMS 2.2A PEAK" (at 158.4 116.1) (layer "F.SilkS")
     (effects (font (size 1 0.6) (thickness 0.15) bold))
   )
-  (gr_text "https://github.com/janelia-kicad/tmc51x0-multiplexer-uart" (at 152.4 119.6) (layer "F.SilkS")
+  (gr_text "https://github.com/janelia-kicad/tmc5130-uart-multiplexer" (at 152.4 119.6) (layer "F.SilkS")
     (effects (font (size 1 0.6) (thickness 0.15) bold))
   )
