File: tmc5130-uart-multiplexer/microcontroller.kicad_sch (KiCad schematic)
At the start: 2 parts

Commit message: Fix some design rule checks
Connections:
- net ENABLE_TX_7: no longer names the net of A401.31 (I2C1-SDA/ADC0/GP26)
- net ~{ENABLE_RX_7}: no longer names the net of A401.32 (I2C1-SCL/ADC1/GP27)
- no-connect marks 12 -> 14
Changed lines of the file:
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@@
   (no_connect (at 180.34 99.06))
   (no_connect (at 93.98 86.36))
+  (no_connect (at 180.34 91.44))
   (no_connect (at 180.34 68.58))
   (no_connect (at 180.34 86.36))
@@
   (no_connect (at 180.34 76.2))
   (no_connect (at 93.98 99.06))
+  (no_connect (at 180.34 88.9))
   (no_connect (at 93.98 73.66))
   (no_connect (at 93.98 111.76))
@@
     (stroke (width 0) (type default))
   )
-  (wire (pts (xy 182.88 91.44) (xy 180.34 91.44))
-    (stroke (width 0) (type default))
-  )
   (wire (pts (xy 180.34 73.66) (xy 182.88 73.66))
-    (stroke (width 0) (type default))
-  )
-  (wire (pts (xy 182.88 88.9) (xy 180.34 88.9))
     (stroke (width 0) (type default))
   )
@@
     (effects (font (size 1.27 1.27)) (justify right))
   )
-  (hierarchical_label "~{ENABLE_RX_7}" (shape output) (at 182.88 88.9 0) (fields_autoplaced)
-    (effects (font (size 1.27 1.27)) (justify left))
-  )
   (hierarchical_label "~{ENABLE_RX_6}" (shape output) (at 91.44 116.84 180) (fields_autoplaced)
     (effects (font (size 1.27 1.27)) (justify right))
@@
     (effects (font (size 1.27 1.27)) (justify right))
   )
-  (hierarchical_label "ENABLE_TX_7" (shape output) (at 182.88 91.44 0) (fields_autoplaced)
-    (effects (font (size 1.27 1.27)) (justify left))
-  )
   (hierarchical_label "+3.3V" (shape passive) (at 54.61 49.53 180) (fields_autoplaced)
