File: honeycomb-pcb/assembly.kicad_sch (KiCad schematic)
At the start: 8 parts

Commit message: tmc5130-uart-multiplexer -> honeycomb-pcb
Other:
- title: tmc5130-uart-multiplexer -> honeycomb-pcb
Changed lines of the file:
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@@
   (paper "A4")
   (title_block
-    (title "tmc5130-uart-multiplexer")
+    (title "honeycomb-pcb")
     (date "2024-07-10")
     (rev "1.0")
@@
     (pin "1")
     (instances
-      (project "tmc5130-uart-multiplexer"
+      (project "honeycomb-pcb"
         (path "/df2b2e89-e055-4140-95de-f1df723db034/0ec4fe58-7f94-4826-b0e2-2bc8f3ffe81e"
           (reference "H201") (unit 1)
@@
     )
     (instances
-      (project "tmc5130-uart-multiplexer"
+      (project "honeycomb-pcb"
         (path "/df2b2e89-e055-4140-95de-f1df723db034/0ec4fe58-7f94-4826-b0e2-2bc8f3ffe81e"
           (reference "FID202") (unit 1)
@@
     (pin "1")
     (instances
-      (project "tmc5130-uart-multiplexer"
+      (project "honeycomb-pcb"
         (path "/df2b2e89-e055-4140-95de-f1df723db034/0ec4fe58-7f94-4826-b0e2-2bc8f3ffe81e"
           (reference "H204") (unit 1)
@@
     (pin "1")
     (instances
-      (project "tmc5130-uart-multiplexer"
+      (project "honeycomb-pcb"
         (path "/df2b2e89-e055-4140-95de-f1df723db034/0ec4fe58-7f94-4826-b0e2-2bc8f3ffe81e"
           (reference "H203") (unit 1)
@@
     )
     (instances
-      (project "tmc5130-uart-multiplexer"
+      (project "honeycomb-pcb"
         (path "/df2b2e89-e055-4140-95de-f1df723db034/0ec4fe58-7f94-4826-b0e2-2bc8f3ffe81e"
           (reference "FID204") (unit 1)
@@
     )
     (instances
-      (project "tmc5130-uart-multiplexer"
+      (project "honeycomb-pcb"
         (path "/df2b2e89-e055-4140-95de-f1df723db034/0ec4fe58-7f94-4826-b0e2-2bc8f3ffe81e"
           (reference "FID201") (unit 1)
@@
     (pin "1")
     (instances
-      (project "tmc5130-uart-multiplexer"
+      (project "honeycomb-pcb"
         (path "/df2b2e89-e055-4140-95de-f1df723db034/0ec4fe58-7f94-4826-b0e2-2bc8f3ffe81e"
           (reference "H202") (unit 1)
@@
     )
     (instances
-      (project "tmc5130-uart-multiplexer"
+      (project "honeycomb-pcb"
         (path "/df2b2e89-e055-4140-95de-f1df723db034/0ec4fe58-7f94-4826-b0e2-2bc8f3ffe81e"
           (reference "FID203") (unit 1)
