File: honeycomb-pcb/microcontroller.kicad_sch (KiCad schematic)
At the start: 2 parts

Commit message: motor -> prism
Other:
- company: (none) -> Howard Hughes Medical Institute
- title: (none) -> honeycomb-pcb
Changed lines of the file:
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@@
 (kicad_sch (version 20230121) (generator eeschema)
   (paper "A4")
+  (title_block
+    (title "honeycomb-pcb")
+    (date "2024-07-12")
+    (rev "1.0")
+    (company "Howard Hughes Medical Institute")
+  )
   (no_connect (at 180.34 81.28))
   (no_connect (at 180.34 99.06))
@@
   (no_connect (at 93.98 111.76))
   (no_connect (at 180.34 83.82))
+  (wire (pts (xy 207.01 46.99) (xy 207.01 49.53))
+    (stroke (width 0) (type default))
+  )
   (wire (pts (xy 91.44 109.22) (xy 93.98 109.22))
     (stroke (width 0) (type default))
@@
     (stroke (width 0) (type default))
   )
+  (wire (pts (xy 195.58 46.99) (xy 195.58 49.53))
+    (stroke (width 0) (type default))
+  )
   (wire (pts (xy 91.44 104.14) (xy 93.98 104.14))
     (stroke (width 0) (type default))
@@
   (label "+3.3V" (at 182.88 78.74 0) (fields_autoplaced)
     (effects (font (size 1.27 1.27)) (justify left bottom))
+  )
+  (label "+3.3V" (at 207.01 49.53 270) (fields_autoplaced)
+    (effects (font (size 1.27 1.27)) (justify right bottom))
   )
   (label "+5V" (at 133.35 58.42 180) (fields_autoplaced)
@@
   (label "+5V" (at 57.15 46.99 0) (fields_autoplaced)
     (effects (font (size 1.27 1.27)) (justify left bottom))
+  )
+  (label "VSYS" (at 195.58 49.53 270) (fields_autoplaced)
+    (effects (font (size 1.27 1.27)) (justify right bottom))
   )
   (label "GND" (at 57.15 52.07 0) (fields_autoplaced)
@@
         )
       )
+    )
+  )
+  (symbol (lib_id "power:PWR_FLAG") (at 195.58 46.99 0) (unit 1)
+    (in_bom yes) (on_board yes) (dnp no)
+    (property "Reference" "#FLG0401" (at 195.58 45.085 0)
+      (effects (font (size 1.27 1.27)) hide)
+    )
+    (property "Value" "PWR_FLAG" (at 195.58 43.18 0)
+      (effects (font (size 1.27 1.27)))
+    )
+    (property "Footprint" "" (at 195.58 46.99 0)
+      (effects (font (size 1.27 1.27)) hide)
+    )
+    (property "Datasheet" "~" (at 195.58 46.99 0)
+      (effects (font (size 1.27 1.27)) hide)
+    )
+    (pin "1")
+    (instances
+      (project "honeycomb-pcb"
+        (path "/df2b2e89-e055-4140-95de-f1df723db034/90ad6836-1738-4b32-a341-0a0b169f4662"
+          (reference "#FLG0401") (unit 1)
+        )
+      )
+    )
+  )
+  (symbol (lib_id "power:PWR_FLAG") (at 207.01 46.99 0) (unit 1)
+    (in_bom yes) (on_board yes) (dnp no)
+    (property "Reference" "#FLG0402" (at 207.01 45.085 0)
+      (effects (font (size 1.27 1.27)) hide)
+    )
+    (property "Value" "PWR_FLAG" (at 207.01 43.18 0)
+      (effects (font (size 1.27 1.27)))
+    )
+    (property "Footprint" "" (at 207.01 46.99 0)
+      (effects (font (size 1.27 1.27)) hide)
+    )
+    (property "Datasheet" "~" (at 207.01 46.99 0)
+      (effects (font (size 1.27 1.27)) hide)
+    )
+    (pin "1")
+    (instances
+      (project "honeycomb-pcb"
+        (path "/df2b2e89-e055-4140-95de-f1df723db034/90ad6836-1738-4b32-a341-0a0b169f4662"
+          (reference "#FLG0402") (unit 1)
+        )
+      )

Commit message: Last update before renaming
Parts:
- D401: Package SOD123FL -> SOD-123FL
Changed lines of the file:
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@@
       (effects (font (size 1.27 1.27)) hide)
     )
-    (property "Package" " SOD123FL" (at 138.43 58.42 0)
+    (property "Package" "SOD-123FL" (at 138.43 58.42 0)
       (effects (font (size 1.27 1.27)) hide)
     )
