File: cluster-pcb/cluster-pcb.kicad_pcb (KiCad board)
At the start: 4 copper layers, 40 x 40 mm, 78 parts, among them J1001 FFC_P1mm_BOT_RA_SMD, J1101 FFC_P1mm_BOT_RA_SMD, J501 FFC_P1mm_BOT_RA_SMD, J601 FFC_P1mm_BOT_RA_SMD, J701 FFC_P1mm_BOT_RA_SMD, J801 FFC_P1mm_BOT_RA_SMD, J901 FFC_P1mm_BOT_RA_SMD, M301 Fan_5VDC_25x25x8mm, Q301 MOSFET-P-CH-EN_60V_50A, Q302 MOSFET-N-CH-EN_100V_260mA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

Commit message: Initial layout
Parts:
- A401: footprint Janelia:Pico_Header_Holes -> Janelia:Pico-W5500-EVB_Header_Holes
- D1001, D1101, D501, D601, D701, D801, D901: value D -> D_Zener_47V_1W; footprint Janelia:D_SMB -> Janelia:D_SMA
- D1002, D1102, D502, D602, D702, D802, D902: value D_Zener_47V_1W -> D; footprint Janelia:D_SMA -> Janelia:D_SMB
- Q301: value MOSFET-P-CH-EN_60V_50A -> MOSFET-N-CH-EN_100V_260mA; footprint Janelia:TO-252-2 -> Janelia:SOT-23
- Q302: value MOSFET-N-CH-EN_100V_260mA -> MOSFET-P-CH-EN_60V_50A; footprint Janelia:SOT-23 -> Janelia:TO-252-2
- moved R701 470.9 mm to (113.4, 80.6), turned to 0 degrees
- moved R801 444.5 mm to (113.4, 100.6), turned to 0 degrees
- moved U1101 435.2 mm to (122.4, 156.6), turned to 0 degrees
- moved R1001 422.0 mm to (113.4, 120.6), turned to 0 degrees
- moved R901 420.6 mm to (113.4, 140.6), turned to 0 degrees
- moved R1101 401.0 mm to (113.4, 160.6), turned to 0 degrees
- moved R501 320.5 mm to (113.4, 40.6), turned to 0 degrees
- moved D902 305.2 mm to (121.4, 144.6), turned to 180 degrees
- moved T301 297.7 mm to (48.2, 55.6), turned to 180 degrees
- moved R902 297.3 mm to (125.4, 136.6), turned to 90 degrees
- moved C901 297.2 mm to (121.4, 133.6)
- moved J901 296.8 mm to (127.4, 141.6), turned to -90 degrees
- moved D901 295.8 mm to (121.4, 140.6)
- moved C902 294.7 mm to (123.4, 133.6), turned to 180 degrees
- moved U901 289.0 mm to (122.4, 136.6), turned to 0 degrees
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Connections:
- net /prism0/SWN renamed /prism-0/SWN
- net /prism0/SWP renamed /prism-0/SWP
- net /prism1/SWN renamed /prism-1/SWN
- net /prism1/SWP renamed /prism-1/SWP
- net /prism2/SWN renamed /prism-2/SWN
- net /prism2/SWP renamed /prism-2/SWP
- net /prism3/SWN renamed /prism-3/SWN
- net /prism3/SWP renamed /prism-3/SWP
- net /prism4/SWN renamed /prism-4/SWN
- net /prism4/SWP renamed /prism-4/SWP
- net /prism5/SWN renamed /prism-5/SWN
- net /prism5/SWP renamed /prism-5/SWP
- net /prism6/SWN renamed /prism-6/SWN
- net /prism6/SWP renamed /prism-6/SWP
- D1001 pad 1: /prism4/VCC -> /prism-4/VBB
- D1001 pad 2: /prism4/VBB -> /GND
- D1002 pad 1: /prism4/VBB -> /prism-4/VCC
- D1002 pad 2: /GND -> /prism-4/VBB
- D1101 pad 1: /prism6/VCC -> /prism-6/VBB
- D1101 pad 2: /prism6/VBB -> /GND
- D1102 pad 1: /prism6/VBB -> /prism-6/VCC
- D1102 pad 2: /GND -> /prism-6/VBB
- D501 pad 1: /prism0/VCC -> /prism-0/VBB
- D501 pad 2: /prism0/VBB -> /GND
- D502 pad 1: /prism0/VBB -> /prism-0/VCC
- D502 pad 2: /GND -> /prism-0/VBB
- D601 pad 1: /prism1/VCC -> /prism-1/VBB
- D601 pad 2: /prism1/VBB -> /GND
- D602 pad 1: /prism1/VBB -> /prism-1/VCC
- D602 pad 2: /GND -> /prism-1/VBB
- D701 pad 1: /prism2/VCC -> /prism-2/VBB
- D701 pad 2: /prism2/VBB -> /GND
- D702 pad 1: /prism2/VBB -> /prism-2/VCC
- D702 pad 2: /GND -> /prism-2/VBB
- D801 pad 1: /prism3/VCC -> /prism-3/VBB
- D801 pad 2: /prism3/VBB -> /GND
- D802 pad 1: /prism3/VBB -> /prism-3/VCC
- D802 pad 2: /GND -> /prism-3/VBB
- D901 pad 1: /prism5/VCC -> /prism-5/VBB
- D901 pad 2: /prism5/VBB -> /GND
- D902 pad 1: /prism5/VBB -> /prism-5/VCC
- D902 pad 2: /GND -> /prism-5/VBB
- J1001 pad 1: /prism4/VCC -> /prism-4/VCC
- J1001 pad 2: /prism4/VCC -> /prism-4/VCC
- J1001 pad 3: /prism4/VCC -> /prism-4/VCC
- J1001 pad 4: /prism4/VCC -> /prism-4/VCC
- J1101 pad 1: /prism6/VCC -> /prism-6/VCC
- J1101 pad 2: /prism6/VCC -> /prism-6/VCC
- J1101 pad 3: /prism6/VCC -> /prism-6/VCC
- J1101 pad 4: /prism6/VCC -> /prism-6/VCC
- J501 pad 1: /prism0/VCC -> /prism-0/VCC
- J501 pad 2: /prism0/VCC -> /prism-0/VCC
- J501 pad 3: /prism0/VCC -> /prism-0/VCC
- J501 pad 4: /prism0/VCC -> /prism-0/VCC
- J601 pad 1: /prism1/VCC -> /prism-1/VCC
- J601 pad 2: /prism1/VCC -> /prism-1/VCC
- J601 pad 3: /prism1/VCC -> /prism-1/VCC
- J601 pad 4: /prism1/VCC -> /prism-1/VCC
- J701 pad 1: /prism2/VCC -> /prism-2/VCC
- J701 pad 2: /prism2/VCC -> /prism-2/VCC
- J701 pad 3: /prism2/VCC -> /prism-2/VCC
- J701 pad 4: /prism2/VCC -> /prism-2/VCC
- J801 pad 1: /prism3/VCC -> /prism-3/VCC
- J801 pad 2: /prism3/VCC -> /prism-3/VCC
- J801 pad 3: /prism3/VCC -> /prism-3/VCC
- J801 pad 4: /prism3/VCC -> /prism-3/VCC
- J901 pad 1: /prism5/VCC -> /prism-5/VCC
- J901 pad 2: /prism5/VCC -> /prism-5/VCC
- J901 pad 3: /prism5/VCC -> /prism-5/VCC
- J901 pad 4: /prism5/VCC -> /prism-5/VCC
- Q301 pad 1: /power/~{ENABLE_VCC} -> /ENABLE_VCC
- Q301 pad 2: /VCC -> /GND
- Q301 pad 3: /power/VBB -> Net-(Q301-D)
- Q302 pad 1: /ENABLE_VCC -> /power/~{ENABLE_VCC}
- Q302 pad 2: /GND -> /VCC
- Q302 pad 3: Net-(Q302-D) -> /power/VBB
- R1001 pad 2: /prism4/VBB -> /prism-4/VBB
- R1101 pad 2: /prism6/VBB -> /prism-6/VBB
- R302 pad 2: Net-(Q302-D) -> Net-(Q301-D)
- R501 pad 2: /prism0/VBB -> /prism-0/VBB
- R601 pad 2: /prism1/VBB -> /prism-1/VBB
- R701 pad 2: /prism2/VBB -> /prism-2/VBB
- R801 pad 2: /prism3/VBB -> /prism-3/VBB
- R901 pad 2: /prism5/VBB -> /prism-5/VBB
Other:
- board size 40 x 40 mm -> 60 x 140 mm

Commit message: Initial layout
Parts:
- removed M301: Fan_5VDC_25x25x8mm, Janelia:FAN_5VDC_25x25x8mm
- C301, C302, D401, FID201, FID203, U301: moved to F.Cu
- moved C301 420.4 mm to (92.4, 101.6), turned to 0 degrees
- moved D401 411.0 mm to (80.4, 94.6)
- moved Q301 410.9 mm to (79.4, 66.6)
- moved R302 408.4 mm to (76.4, 66.6), turned to 0 degrees
- moved R301 401.9 mm to (109.4, 34.6), turned to 0 degrees
- moved C303 390.2 mm to (94.4, 107.6)
- moved C304 377.8 mm to (94.4, 109.6)
- moved D301 373.9 mm to (121.4, 27.6), turned to 0 degrees
- moved U301 266.7 mm to (90.4, 108.6)
- moved C302 252.0 mm to (92.4, 104.6), turned to 0 degrees
- moved Q302 240.1 mm to (109.4, 41.6), turned to -90 degrees
- moved FID203 90.0 mm to (127.4, 171.6), turned to 0 degrees
- moved FID202 80.0 mm to (127.4, 31.6)
- moved T301 78.3 mm to (118.2, 20.6)
- moved FID204 21.2 mm to (77.4, 171.6)
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Other:
- board size 60 x 140 mm -> 60 x 160 mm
