File: cluster-pcb/cluster-pcb.kicad_pcb (KiCad board)
At the start: 4 copper layers, 60 x 160 mm, 77 parts, among them J1001 FFC_P1mm_BOT_RA_SMD, J1101 FFC_P1mm_BOT_RA_SMD, J501 FFC_P1mm_BOT_RA_SMD, J601 FFC_P1mm_BOT_RA_SMD, J701 FFC_P1mm_BOT_RA_SMD, J801 FFC_P1mm_BOT_RA_SMD, J901 FFC_P1mm_BOT_RA_SMD, Q301 MOSFET-N-CH-EN_100V_260mA, Q302 MOSFET-P-CH-EN_60V_50A, T301 TERM_BLK_HDR_2POS_90DEG_0.2IN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

Commit message: Add tracks
Parts:
- moved C301 66.7 mm to (77.4, 36.6)
- moved C302 66.7 mm to (77.4, 39.6)
- moved C303 66.5 mm to (80.4, 42.6)
- moved C304 66.5 mm to (80.4, 44.6)
- moved U301 66.5 mm to (76.4, 43.6)
- moved R302 4.24 mm to (79.4, 63.6), turned to -90 degrees
- moved R1001 2.00 mm to (113.4, 122.6)
- moved R1101 2.00 mm to (113.4, 162.6)
- moved R601 2.00 mm to (113.4, 62.6)
- moved R701 2.00 mm to (113.4, 82.6)
- moved R801 2.00 mm to (113.4, 102.6)
- moved R901 2.00 mm to (113.4, 142.6)
Routing:
- net /GND: track 0.00 -> 177.6 mm, vias 0 -> 28
- net /VCC: track 0.00 -> 120.2 mm
- net /power/VBB: track 0.00 -> 58.4 mm
- net /prism-0/VCC: track 0.00 -> 17.1 mm
- net /prism-6/VCC: track 0.00 -> 17.1 mm
- net /prism-5/VCC: track 0.00 -> 17.1 mm
- net /prism-4/VCC: track 0.00 -> 17.1 mm
- net /prism-3/VCC: track 0.00 -> 17.1 mm
- net /prism-2/VCC: track 0.00 -> 17.1 mm
- net /prism-1/VCC: track 0.00 -> 17.1 mm
- net /prism-0/VBB: track 0.00 -> 9.26 mm
- net /power/VAA: track 0.00 -> 7.69 mm
- net /prism-4/VBB: track 0.00 -> 7.10 mm
- net /prism-3/VBB: track 0.00 -> 7.10 mm
- net /prism-2/VBB: track 0.00 -> 7.10 mm
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
Commit message: Add some more traces
Routing:
- net /+5V: track 7.04 -> 21.2 mm, vias 1 -> 7
- net /+3.3V: track 7.04 -> 21.2 mm, vias 1 -> 7
- net /prism-4/SWP: track 0.00 -> 4.12 mm
- net /prism-4/SWN: track 0.00 -> 3.92 mm
- net /RX: track 1.50 -> 4.50 mm, vias 1 -> 3
- net /TX: track 1.00 -> 3.00 mm, vias 1 -> 3
- net /~{ENABLE_RX_5}: track 0.00 -> 1.50 mm, vias 0 -> 1
- net /~{ENABLE_RX_4}: track 0.00 -> 1.50 mm, vias 0 -> 1
- net /ENABLE_TX_5: track 0.00 -> 1.00 mm, vias 0 -> 1
- net /ENABLE_TX_4: track 0.00 -> 1.00 mm, vias 0 -> 1
Changed lines of the file:
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@@
   (via (at 125.9 161.1) (size 0.75) (drill 0.25) (layers "F.Cu" "B.Cu") (net 1))
   (via (at 125.9 60.1) (size 0.75) (drill 0.25) (layers "F.Cu" "B.Cu") (net 1))
+  (segment (start 120.9014 137.600001) (end 119.9 137.6) (width 0.3) (layer "F.Cu") (net 7))
+  (segment (start 120.9014 117.600001) (end 119.9 117.6) (width 0.3) (layer "F.Cu") (net 7))
   (segment (start 120.9014 157.600001) (end 119.9 157.6) (width 0.3) (layer "F.Cu") (net 7))
+  (via (at 119.9 137.6) (size 0.4) (drill 0.2) (layers "F.Cu" "B.Cu") (net 7))
+  (via (at 119.9 117.6) (size 0.4) (drill 0.2) (layers "F.Cu" "B.Cu") (net 7))
   (via (at 119.9 157.6) (size 0.4) (drill 0.2) (layers "F.Cu" "B.Cu") (net 7))
+  (segment (start 120.9014 116.100001) (end 119.4 116.1) (width 0.3) (layer "F.Cu") (net 8))
   (segment (start 120.9014 156.100001) (end 119.4 156.1) (width 0.3) (layer "F.Cu") (net 8))
+  (segment (start 120.9014 136.100001) (end 119.4 136.1) (width 0.3) (layer "F.Cu") (net 8))
+  (via (at 119.4 136.1) (size 0.4) (drill 0.2) (layers "F.Cu" "B.Cu") (net 8))
+  (via (at 119.4 116.1) (size 0.4) (drill 0.2) (layers "F.Cu" "B.Cu") (net 8))
   (via (at 119.4 156.1) (size 0.4) (drill 0.2) (layers "F.Cu" "B.Cu") (net 8))
+  (segment (start 120.9014 116.6) (end 119.9 116.6) (width 0.3) (layer "F.Cu") (net 15))
+  (via (at 119.9 116.6) (size 0.4) (drill 0.2) (layers "F.Cu" "B.Cu") (net 15))
+  (segment (start 120.9014 117.099999) (end 119.4 117.1) (width 0.3) (layer "F.Cu") (net 16))
+  (via (at 119.4 117.1) (size 0.4) (drill 0.2) (layers "F.Cu" "B.Cu") (net 16))
+  (segment (start 120.9014 136.6) (end 119.9 136.6) (width 0.3) (layer "F.Cu") (net 17))
+  (via (at 119.9 136.6) (size 0.4) (drill 0.2) (layers "F.Cu" "B.Cu") (net 17))
+  (segment (start 120.9014 137.099999) (end 119.4 137.1) (width 0.3) (layer "F.Cu") (net 18))
+  (via (at 119.4 137.1) (size 0.4) (drill 0.2) (layers "F.Cu" "B.Cu") (net 18))
   (segment (start 120.9014 156.6) (end 119.9 156.6) (width 0.3) (layer "F.Cu") (net 20))
   (via (at 119.9 156.6) (size 0.4) (drill 0.2) (layers "F.Cu" "B.Cu") (net 20))
   (segment (start 120.9014 157.099999) (end 119.4 157.1) (width 0.3) (layer "F.Cu") (net 21))
   (via (at 119.4 157.1) (size 0.4) (drill 0.2) (layers "F.Cu" "B.Cu") (net 21))
+  (segment (start 123.88 53.6) (end 124.9 53.6) (width 0.3) (layer "F.Cu") (net 34))
   (segment (start 123.88 153.6) (end 124.9 153.6) (width 0.3) (layer "F.Cu") (net 34))
+  (segment (start 123.88 93.6) (end 124.9 93.6) (width 0.3) (layer "F.Cu") (net 34))
+  (segment (start 123.88 33.6) (end 124.9 33.6) (width 0.3) (layer "F.Cu") (net 34))
+  (segment (start 123.88 133.6) (end 124.9 133.6) (width 0.3) (layer "F.Cu") (net 34))
   (segment (start 123.8986 155.599999) (end 123.8986 153.6186) (width 0.3) (layer "F.Cu") (net 34))
+  (segment (start 123.8986 113.6186) (end 123.88 113.6) (width 0.3) (layer "F.Cu") (net 34))
   (segment (start 123.8986 55.599999) (end 123.8986 53.6186) (width 0.3) (layer "F.Cu") (net 34))
+  (segment (start 123.8986 93.6186) (end 123.88 93.6) (width 0.3) (layer "F.Cu") (net 34))
   (segment (start 123.8986 35.599999) (end 123.8986 33.6186) (width 0.3) (layer "F.Cu") (net 34))
+  (segment (start 123.8986 95.599999) (end 123.8986 93.6186) (width 0.3) (layer "F.Cu") (net 34))
+  (segment (start 123.8986 133.6186) (end 123.88 133.6) (width 0.3) (layer "F.Cu") (net 34))
+  (segment (start 123.88 73.6) (end 124.9 73.6) (width 0.3) (layer "F.Cu") (net 34))
+  (segment (start 123.8986 75.599999) (end 123.8986 73.6186) (width 0.3) (layer "F.Cu") (net 34))
+  (segment (start 123.88 113.6) (end 124.9 113.6) (width 0.3) (layer "F.Cu") (net 34))
   (segment (start 123.8986 53.6186) (end 123.88 53.6) (width 0.3) (layer "F.Cu") (net 34))
+  (segment (start 123.8986 115.599999) (end 123.8986 113.6186) (width 0.3) (layer "F.Cu") (net 34))
+  (segment (start 123.8986 73.6186) (end 123.88 73.6) (width 0.3) (layer "F.Cu") (net 34))
   (segment (start 123.8986 153.6186) (end 123.88 153.6) (width 0.3) (layer "F.Cu") (net 34))
+  (segment (start 123.8986 135.599999) (end 123.8986 133.6186) (width 0.3) (layer "F.Cu") (net 34))
   (segment (start 123.8986 33.6186) (end 123.88 33.6) (width 0.3) (layer "F.Cu") (net 34))
   (via (at 124.9 153.6) (size 0.75) (drill 0.25) (layers "F.Cu" "B.Cu") (net 34))
+  (via (at 124.9 133.6) (size 0.75) (drill 0.25) (layers "F.Cu" "B.Cu") (net 34))
+  (via (at 124.9 33.6) (size 0.75) (drill 0.25) (layers "F.Cu" "B.Cu") (net 34))
+  (via (at 124.9 93.6) (size 0.75) (drill 0.25) (layers "F.Cu" "B.Cu") (net 34))
+  (via (at 124.9 53.6) (size 0.75) (drill 0.25) (layers "F.Cu" "B.Cu") (net 34))
+  (via (at 124.9 113.6) (size 0.75) (drill 0.25) (layers "F.Cu" "B.Cu") (net 34))
+  (via (at 124.9 73.6) (size 0.75) (drill 0.25) (layers "F.Cu" "B.Cu") (net 34))
+  (segment (start 120.9014 113.6186) (end 120.92 113.6) (width 0.3) (layer "F.Cu") (net 38))
+  (segment (start 120.9014 93.6186) (end 120.92 93.6) (width 0.3) (layer "F.Cu") (net 38))
   (segment (start 120.9014 153.6186) (end 120.92 153.6) (width 0.3) (layer "F.Cu") (net 38))
   (segment (start 120.92 153.6) (end 119.9 153.6) (width 0.3) (layer "F.Cu") (net 38))
+  (segment (start 120.92 33.6) (end 119.9 33.6) (width 0.3) (layer "F.Cu") (net 38))
+  (segment (start 120.92 73.6) (end 119.9 73.6) (width 0.3) (layer "F.Cu") (net 38))
+  (segment (start 120.9014 75.599999) (end 120.9014 73.6186) (width 0.3) (layer "F.Cu") (net 38))
   (segment (start 120.9014 35.599999) (end 120.9014 33.6186) (width 0.3) (layer "F.Cu") (net 38))
+  (segment (start 120.92 133.6) (end 119.9 133.6) (width 0.3) (layer "F.Cu") (net 38))
+  (segment (start 120.9014 95.599999) (end 120.9014 93.6186) (width 0.3) (layer "F.Cu") (net 38))
   (segment (start 120.9014 53.6186) (end 120.92 53.6) (width 0.3) (layer "F.Cu") (net 38))
   (segment (start 120.9014 33.6186) (end 120.92 33.6) (width 0.3) (layer "F.Cu") (net 38))
   (segment (start 120.9014 155.599999) (end 120.9014 153.6186) (width 0.3) (layer "F.Cu") (net 38))
+  (segment (start 120.92 113.6) (end 119.9 113.6) (width 0.3) (layer "F.Cu") (net 38))
+  (segment (start 120.9014 73.6186) (end 120.92 73.6) (width 0.3) (layer "F.Cu") (net 38))
+  (segment (start 120.92 53.6) (end 119.9 53.6) (width 0.3) (layer "F.Cu") (net 38))
+  (segment (start 120.9014 115.599999) (end 120.9014 113.6186) (width 0.3) (layer "F.Cu") (net 38))
+  (segment (start 120.92 93.6) (end 119.9 93.6) (width 0.3) (layer "F.Cu") (net 38))
+  (segment (start 120.9014 135.599999) (end 120.9014 133.6186) (width 0.3) (layer "F.Cu") (net 38))
   (segment (start 120.9014 55.599999) (end 120.9014 53.6186) (width 0.3) (layer "F.Cu") (net 38))
+  (segment (start 120.9014 133.6186) (end 120.92 133.6) (width 0.3) (layer "F.Cu") (net 38))
+  (via (at 119.9 33.6) (size 0.75) (drill 0.25) (layers "F.Cu" "B.Cu") (net 38))
+  (via (at 119.9 53.6) (size 0.75) (drill 0.25) (layers "F.Cu" "B.Cu") (net 38))
+  (via (at 119.9 113.6) (size 0.75) (drill 0.25) (layers "F.Cu" "B.Cu") (net 38))
+  (via (at 119.9 93.6) (size 0.75) (drill 0.25) (layers "F.Cu" "B.Cu") (net 38))
+  (via (at 119.9 133.6) (size 0.75) (drill 0.25) (layers "F.Cu" "B.Cu") (net 38))
   (via (at 119.9 153.6) (size 0.75) (drill 0.25) (layers "F.Cu" "B.Cu") (net 38))
+  (via (at 119.9 73.6) (size 0.75) (drill 0.25) (layers "F.Cu" "B.Cu") (net 38))
   (segment (start 107.12 36.56) (end 107.12 30.38) (width 0.6) (layer "F.Cu") (net 42))
   (segment (start 107.12 36.56) (end 104.1925 33.6325) (width 0.6) (layer "F.Cu") (net 42))
@@
   (segment (start 127.4 137.099998) (end 126.409998 137.099998) (width 0.3) (layer "F.Cu") (net 68))
   (segment (start 126.409998 137.099998) (end 125.4 136.09) (width 0.3) (layer "F.Cu") (net 68))
+  (segment (start 127.4 118.099998) (end 126.389998 118.099998) (width 0.3) (layer "F.Cu") (net 69))
+  (segment (start 124.89 116.6) (end 125.4 117.11) (width 0.3) (layer "F.Cu") (net 69))
+  (segment (start 126.389998 118.099998) (end 125.4 117.11) (width 0.3) (layer "F.Cu") (net 69))
+  (segment (start 123.8986 116.6) (end 124.89 116.6) (width 0.3) (layer "F.Cu") (net 69))
+  (segment (start 123.8986 116.100001) (end 125.389999 116.100001) (width 0.3) (layer "F.Cu") (net 70))
+  (segment (start 125.389999 116.100001) (end 125.4 116.09) (width 0.3) (layer "F.Cu") (net 70))
+  (segment (start 126.409998 117.099998) (end 125.4 116.09) (width 0.3) (layer "F.Cu") (net 70))
+  (segment (start 127.4 117.099998) (end 126.409998 117.099998) (width 0.3) (layer "F.Cu") (net 70))
   (segment (start 126.389998 158.099998) (end 125.4 157.11) (width 0.3) (layer "F.Cu") (net 71))
   (segment (start 123.8986 156.6) (end 124.89 156.6) (width 0.3) (layer "F.Cu") (net 71))

Commit message: Finalize layout
Parts:
- moved FID202 3.61 mm to (130.4, 29.6)
- moved FID203 3.61 mm to (130.4, 173.6)
- moved D401 3.35 mm to (77.4, 93.1), turned to 180 degrees
Connections:
- A401 pad 1: /ENABLE_TX_0 -> /~{ENABLE_RX_6}
- A401 pad 10: /~{ENABLE_RX_2} -> /ENABLE_TX_4
- A401 pad 11: /ENABLE_TX_3 -> /~{ENABLE_RX_3}
- A401 pad 12: /~{ENABLE_RX_3} -> /ENABLE_TX_3
- A401 pad 14: /ENABLE_TX_4 -> /~{ENABLE_RX_2}
- A401 pad 15: /~{ENABLE_RX_4} -> /ENABLE_TX_2
- A401 pad 16: /ENABLE_TX_5 -> /~{ENABLE_RX_1}
- A401 pad 17: /~{ENABLE_RX_5} -> /ENABLE_TX_1
- A401 pad 19: /ENABLE_TX_6 -> /~{ENABLE_RX_0}
- A401 pad 2: /~{ENABLE_RX_0} -> /ENABLE_TX_6
- A401 pad 20: /~{ENABLE_RX_6} -> /ENABLE_TX_0
- A401 pad 4: /ENABLE_TX_1 -> /~{ENABLE_RX_5}
- A401 pad 5: /~{ENABLE_RX_1} -> /ENABLE_TX_5
- A401 pad 9: /ENABLE_TX_2 -> /~{ENABLE_RX_4}
Routing:
- net /GND: track 177.6 -> 631.7 mm, vias 28 -> 31
- net /+5V: track 21.2 -> 263.8 mm, vias 7 -> 9
- net /+3.3V: track 21.2 -> 186.5 mm
- net /RX: track 4.50 -> 150.3 mm, vias 3 -> 7
- net /TX: track 3.00 -> 147.8 mm, vias 3 -> 7
- net /ENABLE_TX_6: track 1.00 -> 77.9 mm
- net /~{ENABLE_RX_6}: track 1.50 -> 76.8 mm
- net /ENABLE_TX_5: track 1.00 -> 62.2 mm
- net /~{ENABLE_RX_5}: track 1.50 -> 61.3 mm
- net /power/~{ENABLE_VCC}: track 0.00 -> 55.0 mm, vias 0 -> 2
- net /ENABLE_TX_4: track 1.00 -> 55.1 mm
- net /~{ENABLE_RX_4}: track 1.50 -> 54.5 mm
- net /VCC: track 120.2 -> 160.5 mm
- net /ENABLE_TX_3: track 0.00 -> 38.4 mm, vias 0 -> 1
- net /~{ENABLE_RX_3}: track 0.00 -> 37.5 mm, vias 0 -> 1
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- added copper zone on B.Cu, net /GND
- added copper zone on In1.Cu, net /GND
- added copper zone on In2.Cu, net /GND
- added copper zone on F.Cu, net /VCC
- added copper zone on F.Cu, net /power/VAA
- added copper zone on F.Cu, net /power/VBB
Other:
- board text added: "+48VDC"
- board text added: "0"
- board text added: "1"
- board text added: "2"
- board text added: "3"
- board text added: "4"
- board text added: "5"
- board text added: "6"
- board text added: "GND"
- board text added: "RX"
- board text added: "TX"
- board text added: "cluster-pcb v1.0 2024/07"
- board text added: "https://github.com/janelia-kicad/cluster-pcb"
