File: cluster-pcb/cluster-pcb.kicad_sch (KiCad schematic)
At the start: 0 parts

Commit message: honeycomb-pcb -> cluster-pcb
Other:
- title: honeycomb-pcb -> cluster-pcb
Changed lines of the file:
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@@
   (paper "A4")
   (title_block
-    (title "honeycomb-pcb")
+    (title "cluster-pcb")
     (date "2024-07-16")
     (rev "1.0")
@@
     )
     (instances
-      (project "honeycomb-pcb"
+      (project "cluster-pcb"
         (path "/df2b2e89-e055-4140-95de-f1df723db034" (page "2"))
       )
@@
     )
     (instances
-      (project "honeycomb-pcb"
+      (project "cluster-pcb"
         (path "/df2b2e89-e055-4140-95de-f1df723db034" (page "5"))
       )
@@
     )
     (instances
-      (project "honeycomb-pcb"
+      (project "cluster-pcb"
         (path "/df2b2e89-e055-4140-95de-f1df723db034" (page "9"))
       )
@@
     )
     (instances
-      (project "honeycomb-pcb"
+      (project "cluster-pcb"
         (path "/df2b2e89-e055-4140-95de-f1df723db034" (page "11"))
       )
@@
     )
     (instances
-      (project "honeycomb-pcb"
+      (project "cluster-pcb"
         (path "/df2b2e89-e055-4140-95de-f1df723db034" (page "4"))
       )
@@
     )
     (instances
-      (project "honeycomb-pcb"
+      (project "cluster-pcb"
         (path "/df2b2e89-e055-4140-95de-f1df723db034" (page "7"))
       )
@@
     )
     (instances
-      (project "honeycomb-pcb"
+      (project "cluster-pcb"
         (path "/df2b2e89-e055-4140-95de-f1df723db034" (page "6"))
       )
@@
     )
     (instances
-      (project "honeycomb-pcb"
+      (project "cluster-pcb"
         (path "/df2b2e89-e055-4140-95de-f1df723db034" (page "10"))
       )
@@
     )
     (instances
-      (project "honeycomb-pcb"
+      (project "cluster-pcb"
         (path "/df2b2e89-e055-4140-95de-f1df723db034" (page "3"))
       )
@@
     )
     (instances
-      (project "honeycomb-pcb"
+      (project "cluster-pcb"
         (path "/df2b2e89-e055-4140-95de-f1df723db034" (page "8"))
       )

Commit message: Initial layout
Other:
- sheet prism0 renamed prism-0
- sheet prism1 renamed prism-1
- sheet prism2 renamed prism-2
- sheet prism3 renamed prism-3
- sheet prism4 renamed prism-4
- sheet prism5 renamed prism-5
- sheet prism6 renamed prism-6
Changed lines of the file:
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@@
     (stroke (width 0.1524) (type solid))
     (fill (color 0 0 0 0.0000))
-    (property "Sheetname" "prism0" (at 135.89 48.8184 0)
+    (property "Sheetname" "prism-0" (at 135.89 48.8184 0)
       (effects (font (size 1.27 1.27)) (justify left bottom))
     )
@@
     (stroke (width 0.1524) (type solid))
     (fill (color 0 0 0 0.0000))
-    (property "Sheetname" "prism5" (at 181.61 78.0284 0)
+    (property "Sheetname" "prism-5" (at 181.61 78.0284 0)
       (effects (font (size 1.27 1.27)) (justify left bottom))
     )
@@
     (stroke (width 0.1524) (type solid))
     (fill (color 0 0 0 0.0000))
-    (property "Sheetname" "prism6" (at 181.61 107.2384 0)
+    (property "Sheetname" "prism-6" (at 181.61 107.2384 0)
       (effects (font (size 1.27 1.27)) (justify left bottom))
     )
@@
     (stroke (width 0.1524) (type solid))
     (fill (color 0 0 0 0.0000))
-    (property "Sheetname" "prism2" (at 135.89 107.2384 0)
+    (property "Sheetname" "prism-2" (at 135.89 107.2384 0)
       (effects (font (size 1.27 1.27)) (justify left bottom))
     )
@@
     (stroke (width 0.1524) (type solid))
     (fill (color 0 0 0 0.0000))
-    (property "Sheetname" "prism1" (at 135.89 78.0284 0)
+    (property "Sheetname" "prism-1" (at 135.89 78.0284 0)
       (effects (font (size 1.27 1.27)) (justify left bottom))
     )
@@
     (stroke (width 0.1524) (type solid))
     (fill (color 0 0 0 0.0000))
-    (property "Sheetname" "prism4" (at 181.61 48.8184 0)
+    (property "Sheetname" "prism-4" (at 181.61 48.8184 0)
       (effects (font (size 1.27 1.27)) (justify left bottom))
     )
@@
     (stroke (width 0.1524) (type solid))
     (fill (color 0 0 0 0.0000))
-    (property "Sheetname" "prism3" (at 135.89 136.4484 0)
-      (effects (font (size 1.27 1.27)) (justify left bottom))
-    )
+    (property "Sheetname" "prism-3" (at 135.89 136.4484 0)
+      (effects (font (size 1.27 1.27)) (justify left bottom))
+    )
