File: cluster-pcb/microcontroller.kicad_sch (KiCad schematic)
At the start: 2 parts

Commit message: honeycomb-pcb -> cluster-pcb
Other:
- title: honeycomb-pcb -> cluster-pcb
Changed lines of the file:
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@@
   (paper "A4")
   (title_block
-    (title "honeycomb-pcb")
+    (title "cluster-pcb")
     (date "2024-07-16")
     (rev "1.0")
@@
     (pin "16")
     (instances
-      (project "honeycomb-pcb"
+      (project "cluster-pcb"
         (path "/df2b2e89-e055-4140-95de-f1df723db034/90ad6836-1738-4b32-a341-0a0b169f4662"
           (reference "A401") (unit 1)
@@
     (pin "1")
     (instances
-      (project "honeycomb-pcb"
+      (project "cluster-pcb"
         (path "/df2b2e89-e055-4140-95de-f1df723db034/90ad6836-1738-4b32-a341-0a0b169f4662"
           (reference "#FLG0401") (unit 1)
@@
     (pin "1")
     (instances
-      (project "honeycomb-pcb"
+      (project "cluster-pcb"
         (path "/df2b2e89-e055-4140-95de-f1df723db034/90ad6836-1738-4b32-a341-0a0b169f4662"
           (reference "#FLG0402") (unit 1)
@@
     (pin "2")
     (instances
-      (project "honeycomb-pcb"
+      (project "cluster-pcb"
         (path "/df2b2e89-e055-4140-95de-f1df723db034/90ad6836-1738-4b32-a341-0a0b169f4662"
           (reference "D401") (unit 1)

Commit message: Initial layout
Parts:
- A401: footprint Janelia:Pico_Header_Holes -> Janelia:Pico-W5500-EVB_Header_Holes
Changed lines of the file:
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@@
       (effects (font (size 1.524 1.524)))
     )
-    (property "Footprint" "Janelia:Pico_Header_Holes" (at 137.16 62.23 0)
+    (property "Footprint" "Janelia:Pico-W5500-EVB_Header_Holes" (at 137.16 62.23 0)
       (effects (font (size 1.524 1.524)) hide)
     )
