File: cluster-pcb/microcontroller.kicad_sch (KiCad schematic)
At the start: 4 parts

Commit message: Progress towards layout
Connections:
- net ~{PRISM_CS_0}: now also A401.11 (UART1-TX/I2C0-SDA/SPI1-RX/GP8); no longer A401.19 (I2C1-SDA/SPI1-SCK/GP14)
- net ~{PRISM_CS_1}: now also A401.10 (I2C1-SCL/SPI0-TX/GP7); no longer A401.17 (UART0-RX/I2C0-SCL/SPI1-CS/GP13)
- net ~{PRISM_CS_2}: now also A401.9 (I2C1-SDA/SPI0-SCK/GP6); no longer A401.12 (UART1-RX/I2C0-SCL/SPI1-CS/GP9)
- net ~{PRISM_CS_3}: now also A401.7 (UART1-RX/I2C0-SCL/SPI0-CS/GP5); no longer A401.11 (UART1-TX/I2C0-SDA/SPI1-RX/GP8)
- net ~{PRISM_CS_4}: now also A401.6 (UART1-TX/I2C0-SDA/SPI0-RX/GP4); no longer A401.10 (I2C1-SCL/SPI0-TX/GP7)
- net ~{PRISM_CS_5}: now also A401.5 (I2C1-SCL/SPI0-TX/GP3); no longer A401.9 (I2C1-SDA/SPI0-SCK/GP6)
- net ~{PRISM_CS_6}: now also A401.4 (I2C1-SDA/SPI0-SCK/GP2); no longer A401.7 (UART1-RX/I2C0-SCL/SPI0-CS/GP5)
Changed lines of the file:
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@@
   (title_block
     (title "cluster-pcb")
-    (date "2024-09-27")
+    (date "2024-09-30")
     (rev "2.0")
     (company "Howard Hughes Medical Institute")
@@
   (no_connect (at 180.34 99.06))
   (no_connect (at 93.98 86.36))
-  (no_connect (at 93.98 76.2))
+  (no_connect (at 93.98 96.52))
   (no_connect (at 180.34 68.58))
   (no_connect (at 180.34 86.36))
@@
   (no_connect (at 180.34 76.2))
   (no_connect (at 180.34 96.52))
-  (no_connect (at 93.98 78.74))
+  (no_connect (at 93.98 109.22))
   (no_connect (at 93.98 99.06))
-  (no_connect (at 93.98 81.28))
+  (no_connect (at 93.98 114.3))
   (no_connect (at 93.98 73.66))
   (no_connect (at 93.98 111.76))
@@
     (stroke (width 0) (type default))
   )
-  (wire (pts (xy 91.44 96.52) (xy 93.98 96.52))
+  (wire (pts (xy 91.44 83.82) (xy 93.98 83.82))
     (stroke (width 0) (type default))
   )
@@
     (stroke (width 0) (type default))
   )
-  (wire (pts (xy 91.44 109.22) (xy 93.98 109.22))
+  (wire (pts (xy 91.44 81.28) (xy 93.98 81.28))
     (stroke (width 0) (type default))
   )
@@
     (stroke (width 0) (type default))
   )
-  (wire (pts (xy 91.44 83.82) (xy 93.98 83.82))
+  (wire (pts (xy 91.44 76.2) (xy 93.98 76.2))
     (stroke (width 0) (type default))
   )
@@
     (stroke (width 0) (type default))
   )
-  (wire (pts (xy 91.44 114.3) (xy 93.98 114.3))
+  (wire (pts (xy 91.44 78.74) (xy 93.98 78.74))
     (stroke (width 0) (type default))
   )
@@
     (effects (font (size 1.27 1.27)) (justify left bottom))
   )
-  (hierarchical_label "~{PRISM_CS_2}" (shape output) (at 91.44 96.52 180) (fields_autoplaced)
+  (hierarchical_label "~{PRISM_CS_2}" (shape output) (at 91.44 88.9 180) (fields_autoplaced)
     (effects (font (size 1.27 1.27)) (justify right))
   )
@@
     (effects (font (size 1.27 1.27)) (justify right))
   )
-  (hierarchical_label "~{PRISM_CS_4}" (shape output) (at 91.44 91.44 180) (fields_autoplaced)
+  (hierarchical_label "~{PRISM_CS_4}" (shape output) (at 91.44 81.28 180) (fields_autoplaced)
     (effects (font (size 1.27 1.27)) (justify right))
   )
@@
     (effects (font (size 1.27 1.27)) (justify right))
   )
-  (hierarchical_label "~{PRISM_CS_1}" (shape output) (at 91.44 109.22 180) (fields_autoplaced)
+  (hierarchical_label "~{PRISM_CS_1}" (shape output) (at 91.44 91.44 180) (fields_autoplaced)
     (effects (font (size 1.27 1.27)) (justify right))
   )
@@
     (effects (font (size 1.27 1.27)) (justify right))
   )
-  (hierarchical_label "~{PRISM_CS_6}" (shape output) (at 91.44 83.82 180) (fields_autoplaced)
+  (hierarchical_label "~{PRISM_CS_6}" (shape output) (at 91.44 76.2 180) (fields_autoplaced)
     (effects (font (size 1.27 1.27)) (justify right))
   )
@@
     (effects (font (size 1.27 1.27)) (justify right))
   )
-  (hierarchical_label "~{PRISM_CS_5}" (shape output) (at 91.44 88.9 180) (fields_autoplaced)
-    (effects (font (size 1.27 1.27)) (justify right))
-  )
-  (hierarchical_label "~{PRISM_CS_3}" (shape output) (at 91.44 93.98 180) (fields_autoplaced)
-    (effects (font (size 1.27 1.27)) (justify right))
-  )
-  (hierarchical_label "~{PRISM_CS_0}" (shape output) (at 91.44 114.3 180) (fields_autoplaced)
-    (effects (font (size 1.27 1.27)) (justify right))
-  )
+  (hierarchical_label "~{PRISM_CS_5}" (shape output) (at 91.44 78.74 180) (fields_autoplaced)
+    (effects (font (size 1.27 1.27)) (justify right))
+  )
+  (hierarchical_label "~{PRISM_CS_3}" (shape output) (at 91.44 83.82 180) (fields_autoplaced)
+    (effects (font (size 1.27 1.27)) (justify right))
+  )
+  (hierarchical_label "~{PRISM_CS_0}" (shape output) (at 91.44 93.98 180) (fields_autoplaced)
+    (effects (font (size 1.27 1.27)) (justify right))
+  )

Commit message: Update routing
Connections:
- net ~{PRISM_CS_0}: now also A401.19 (I2C1-SDA/SPI1-SCK/GP14); no longer A401.11 (UART1-TX/I2C0-SDA/SPI1-RX/GP8)
- net ~{PRISM_CS_1}: now also A401.11 (UART1-TX/I2C0-SDA/SPI1-RX/GP8); no longer A401.10 (I2C1-SCL/SPI0-TX/GP7)
- net ~{PRISM_CS_2}: now also A401.10 (I2C1-SCL/SPI0-TX/GP7); no longer A401.9 (I2C1-SDA/SPI0-SCK/GP6)
- net ~{PRISM_CS_3}: now also A401.9 (I2C1-SDA/SPI0-SCK/GP6); no longer A401.7 (UART1-RX/I2C0-SCL/SPI0-CS/GP5)
- net ~{PRISM_CS_4}: now also A401.7 (UART1-RX/I2C0-SCL/SPI0-CS/GP5); no longer A401.6 (UART1-TX/I2C0-SDA/SPI0-RX/GP4)
- net ~{PRISM_CS_5}: now also A401.6 (UART1-TX/I2C0-SDA/SPI0-RX/GP4); no longer A401.5 (I2C1-SCL/SPI0-TX/GP3)
- net ~{PRISM_CS_6}: now also A401.5 (I2C1-SCL/SPI0-TX/GP3); no longer A401.4 (I2C1-SDA/SPI0-SCK/GP2)
- net ENABLE_POWER renamed ENABLE_PRISMS
Changed lines of the file:
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@@
   )
   (no_connect (at 180.34 81.28))
+  (no_connect (at 93.98 76.2))
   (no_connect (at 180.34 99.06))
   (no_connect (at 93.98 86.36))
@@
   (no_connect (at 93.98 109.22))
   (no_connect (at 93.98 99.06))
-  (no_connect (at 93.98 114.3))
   (no_connect (at 93.98 73.66))
   (no_connect (at 93.98 111.76))
@@
     (stroke (width 0) (type default))
   )
+  (wire (pts (xy 91.44 88.9) (xy 93.98 88.9))
+    (stroke (width 0) (type default))
+  )
+  (wire (pts (xy 91.44 93.98) (xy 93.98 93.98))
+    (stroke (width 0) (type default))
+  )
+  (wire (pts (xy 207.01 46.99) (xy 207.01 49.53))
+    (stroke (width 0) (type default))
+  )
+  (wire (pts (xy 226.06 88.9) (xy 226.06 91.44))
+    (stroke (width 0) (type default))
+  )
   (wire (pts (xy 91.44 83.82) (xy 93.98 83.82))
     (stroke (width 0) (type default))
   )
+  (wire (pts (xy 226.06 76.2) (xy 226.06 73.66))
+    (stroke (width 0) (type default))
+  )
+  (wire (pts (xy 180.34 91.44) (xy 182.88 91.44))
+    (stroke (width 0) (type default))
+  )
+  (wire (pts (xy 58.42 46.99) (xy 60.96 46.99))
+    (stroke (width 0) (type default))
+  )
+  (wire (pts (xy 91.44 104.14) (xy 93.98 104.14))
+    (stroke (width 0) (type default))
+  )
+  (wire (pts (xy 58.42 54.61) (xy 60.96 54.61))
+    (stroke (width 0) (type default))
+  )
+  (wire (pts (xy 91.44 114.3) (xy 93.98 114.3))
+    (stroke (width 0) (type default))
+  )
+  (wire (pts (xy 195.58 46.99) (xy 195.58 49.53))
+    (stroke (width 0) (type default))
+  )
+  (wire (pts (xy 91.44 68.58) (xy 93.98 68.58))
+    (stroke (width 0) (type default))
+  )
+  (wire (pts (xy 180.34 78.74) (xy 182.88 78.74))
+    (stroke (width 0) (type default))
+  )
   (wire (pts (xy 91.44 91.44) (xy 93.98 91.44))
     (stroke (width 0) (type default))
   )
-  (wire (pts (xy 207.01 46.99) (xy 207.01 49.53))
-    (stroke (width 0) (type default))
-  )
-  (wire (pts (xy 226.06 88.9) (xy 226.06 91.44))
+  (wire (pts (xy 58.42 49.53) (xy 60.96 49.53))
+    (stroke (width 0) (type default))
+  )
+  (wire (pts (xy 91.44 116.84) (xy 93.98 116.84))
+    (stroke (width 0) (type default))
+  )
+  (wire (pts (xy 180.34 73.66) (xy 182.88 73.66))
+    (stroke (width 0) (type default))
+  )
+  (wire (pts (xy 91.44 106.68) (xy 93.98 106.68))
+    (stroke (width 0) (type default))
+  )
+  (wire (pts (xy 234.95 88.9) (xy 234.95 91.44))
+    (stroke (width 0) (type default))
+  )
+  (wire (pts (xy 58.42 52.07) (xy 60.96 52.07))
+    (stroke (width 0) (type default))
+  )
+  (wire (pts (xy 140.97 58.42) (xy 143.51 58.42))
+    (stroke (width 0) (type default))
+  )
+  (wire (pts (xy 135.89 58.42) (xy 133.35 58.42))
+    (stroke (width 0) (type default))
+  )
+  (wire (pts (xy 58.42 44.45) (xy 60.96 44.45))
+    (stroke (width 0) (type default))
+  )
+  (wire (pts (xy 180.34 83.82) (xy 182.88 83.82))
+    (stroke (width 0) (type default))
+  )
+  (wire (pts (xy 180.34 88.9) (xy 182.88 88.9))
+    (stroke (width 0) (type default))
+  )
+  (wire (pts (xy 91.44 78.74) (xy 93.98 78.74))
+    (stroke (width 0) (type default))
+  )
+  (wire (pts (xy 180.34 71.12) (xy 182.88 71.12))
+    (stroke (width 0) (type default))
+  )
+  (wire (pts (xy 234.95 76.2) (xy 234.95 73.66))
+    (stroke (width 0) (type default))
+  )
+  (wire (pts (xy 91.44 71.12) (xy 93.98 71.12))
     (stroke (width 0) (type default))
   )
@@
     (stroke (width 0) (type default))
   )
-  (wire (pts (xy 226.06 76.2) (xy 226.06 73.66))
-    (stroke (width 0) (type default))
-  )
-  (wire (pts (xy 180.34 91.44) (xy 182.88 91.44))
-    (stroke (width 0) (type default))
-  )
-  (wire (pts (xy 58.42 46.99) (xy 60.96 46.99))
-    (stroke (width 0) (type default))
-  )
-  (wire (pts (xy 91.44 104.14) (xy 93.98 104.14))
-    (stroke (width 0) (type default))
-  )
-  (wire (pts (xy 58.42 54.61) (xy 60.96 54.61))
-    (stroke (width 0) (type default))
-  )
-  (wire (pts (xy 91.44 93.98) (xy 93.98 93.98))
-    (stroke (width 0) (type default))
-  )
-  (wire (pts (xy 195.58 46.99) (xy 195.58 49.53))
-    (stroke (width 0) (type default))
-  )
-  (wire (pts (xy 91.44 68.58) (xy 93.98 68.58))
-    (stroke (width 0) (type default))
-  )
-  (wire (pts (xy 180.34 78.74) (xy 182.88 78.74))
-    (stroke (width 0) (type default))
-  )
-  (wire (pts (xy 91.44 88.9) (xy 93.98 88.9))
-    (stroke (width 0) (type default))
-  )
-  (wire (pts (xy 58.42 49.53) (xy 60.96 49.53))
-    (stroke (width 0) (type default))
-  )
-  (wire (pts (xy 91.44 116.84) (xy 93.98 116.84))
-    (stroke (width 0) (type default))
-  )
-  (wire (pts (xy 180.34 73.66) (xy 182.88 73.66))
-    (stroke (width 0) (type default))
-  )
-  (wire (pts (xy 91.44 106.68) (xy 93.98 106.68))
-    (stroke (width 0) (type default))
-  )
-  (wire (pts (xy 234.95 88.9) (xy 234.95 91.44))
-    (stroke (width 0) (type default))
-  )
-  (wire (pts (xy 58.42 52.07) (xy 60.96 52.07))
-    (stroke (width 0) (type default))
-  )
-  (wire (pts (xy 140.97 58.42) (xy 143.51 58.42))
-    (stroke (width 0) (type default))
-  )
-  (wire (pts (xy 135.89 58.42) (xy 133.35 58.42))
-    (stroke (width 0) (type default))
-  )
-  (wire (pts (xy 58.42 44.45) (xy 60.96 44.45))
-    (stroke (width 0) (type default))
-  )
-  (wire (pts (xy 180.34 83.82) (xy 182.88 83.82))
-    (stroke (width 0) (type default))
-  )
-  (wire (pts (xy 180.34 88.9) (xy 182.88 88.9))
-    (stroke (width 0) (type default))
-  )
-  (wire (pts (xy 91.44 76.2) (xy 93.98 76.2))
-    (stroke (width 0) (type default))
-  )
-  (wire (pts (xy 180.34 71.12) (xy 182.88 71.12))
-    (stroke (width 0) (type default))
-  )
-  (wire (pts (xy 234.95 76.2) (xy 234.95 73.66))
-    (stroke (width 0) (type default))
-  )
-  (wire (pts (xy 91.44 71.12) (xy 93.98 71.12))
-    (stroke (width 0) (type default))
-  )
-  (wire (pts (xy 91.44 78.74) (xy 93.98 78.74))
-    (stroke (width 0) (type default))
-  )
   (label "+3.3V" (at 60.96 46.99 0) (fields_autoplaced)
     (effects (font (size 1.27 1.27)) (justify left bottom))
@@
     (effects (font (size 1.27 1.27)) (justify left bottom))
   )
-  (hierarchical_label "~{PRISM_CS_2}" (shape output) (at 91.44 88.9 180) (fields_autoplaced)
+  (hierarchical_label "~{PRISM_CS_2}" (shape output) (at 91.44 91.44 180) (fields_autoplaced)
     (effects (font (size 1.27 1.27)) (justify right))
   )
@@
     (effects (font (size 1.27 1.27)) (justify left))
   )
-  (hierarchical_label "ENABLE_POWER" (shape output) (at 91.44 116.84 180) (fields_autoplaced)
+  (hierarchical_label "ENABLE_PRISMS" (shape output) (at 91.44 116.84 180) (fields_autoplaced)
     (effects (font (size 1.27 1.27)) (justify right))
   )
@@
     (effects (font (size 1.27 1.27)) (justify right))
   )
-  (hierarchical_label "~{PRISM_CS_4}" (shape output) (at 91.44 81.28 180) (fields_autoplaced)
+  (hierarchical_label "~{PRISM_CS_4}" (shape output) (at 91.44 83.82 180) (fields_autoplaced)
     (effects (font (size 1.27 1.27)) (justify right))
   )
@@
     (effects (font (size 1.27 1.27)) (justify right))
   )
-  (hierarchical_label "~{PRISM_CS_1}" (shape output) (at 91.44 91.44 180) (fields_autoplaced)
+  (hierarchical_label "~{PRISM_CS_1}" (shape output) (at 91.44 93.98 180) (fields_autoplaced)
     (effects (font (size 1.27 1.27)) (justify right))
   )
@@
     (effects (font (size 1.27 1.27)) (justify right))
   )
-  (hierarchical_label "~{PRISM_CS_6}" (shape output) (at 91.44 76.2 180) (fields_autoplaced)
+  (hierarchical_label "~{PRISM_CS_6}" (shape output) (at 91.44 78.74 180) (fields_autoplaced)
     (effects (font (size 1.27 1.27)) (justify right))
   )
@@
     (effects (font (size 1.27 1.27)) (justify right))
   )
-  (hierarchical_label "~{PRISM_CS_5}" (shape output) (at 91.44 78.74 180) (fields_autoplaced)
-    (effects (font (size 1.27 1.27)) (justify right))
-  )
-  (hierarchical_label "~{PRISM_CS_3}" (shape output) (at 91.44 83.82 180) (fields_autoplaced)
-    (effects (font (size 1.27 1.27)) (justify right))
-  )
-  (hierarchical_label "~{PRISM_CS_0}" (shape output) (at 91.44 93.98 180) (fields_autoplaced)
-    (effects (font (size 1.27 1.27)) (justify right))
-  )
+  (hierarchical_label "~{PRISM_CS_5}" (shape output) (at 91.44 81.28 180) (fields_autoplaced)
+    (effects (font (size 1.27 1.27)) (justify right))
+  )
+  (hierarchical_label "~{PRISM_CS_3}" (shape output) (at 91.44 88.9 180) (fields_autoplaced)
+    (effects (font (size 1.27 1.27)) (justify right))
+  )
+  (hierarchical_label "~{PRISM_CS_0}" (shape output) (at 91.44 114.3 180) (fields_autoplaced)
+    (effects (font (size 1.27 1.27)) (justify right))
+  )

Commit message: Finish routing
Connections:
- net ENABLE_PRISMS renamed ~{PRISMS_RESET}
Changed lines of the file:
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@@
   (title_block
     (title "cluster-pcb")
-    (date "2024-09-30")
+    (date "2024-10-01")
     (rev "2.0")
     (company "Howard Hughes Medical Institute")
@@
     (effects (font (size 1.27 1.27)) (justify left))
   )
-  (hierarchical_label "ENABLE_PRISMS" (shape output) (at 91.44 116.84 180) (fields_autoplaced)
+  (hierarchical_label "~{PRISMS_RESET}" (shape output) (at 91.44 116.84 180) (fields_autoplaced)
     (effects (font (size 1.27 1.27)) (justify right))
   )
