File: cluster-pcb/power.kicad_sch (KiCad schematic)
At the start: 12 parts, among them M301 Fan_5VDC_25x25x8mm, Q301 MOSFET-P-CH-EN_60V_50A, Q302 MOSFET-N-CH-EN_100V_260mA, T301 TERM_BLK_HDR_2POS_90DEG_0.2IN, U301 TPSM365R6V5RDNR

Commit message: honeycomb-pcb -> cluster-pcb
Other:
- title: honeycomb-pcb -> cluster-pcb
Changed lines of the file:
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@@
   (paper "A4")
   (title_block
-    (title "honeycomb-pcb")
+    (title "cluster-pcb")
     (date "2024-07-16")
     (rev "1.0")
@@
     (pin "1")
     (instances
-      (project "honeycomb-pcb"
+      (project "cluster-pcb"
         (path "/df2b2e89-e055-4140-95de-f1df723db034/c1dd8f61-494c-402f-8e59-08309c64fc3f"
           (reference "T301") (unit 1)
@@
     (pin "1")
     (instances
-      (project "honeycomb-pcb"
+      (project "cluster-pcb"
         (path "/df2b2e89-e055-4140-95de-f1df723db034/c1dd8f61-494c-402f-8e59-08309c64fc3f"
           (reference "#FLG0301") (unit 1)
@@
     (pin "1")
     (instances
-      (project "honeycomb-pcb"
+      (project "cluster-pcb"
         (path "/df2b2e89-e055-4140-95de-f1df723db034/c1dd8f61-494c-402f-8e59-08309c64fc3f"
           (reference "C303") (unit 1)
@@
     (pin "1")
     (instances
-      (project "honeycomb-pcb"
+      (project "cluster-pcb"
         (path "/df2b2e89-e055-4140-95de-f1df723db034/c1dd8f61-494c-402f-8e59-08309c64fc3f"
           (reference "Q301") (unit 1)
@@
     (pin "1")
     (instances
-      (project "honeycomb-pcb"
+      (project "cluster-pcb"
         (path "/df2b2e89-e055-4140-95de-f1df723db034/c1dd8f61-494c-402f-8e59-08309c64fc3f"
           (reference "#FLG0305") (unit 1)
@@
     (pin "4")
     (instances
-      (project "honeycomb-pcb"
+      (project "cluster-pcb"
         (path "/df2b2e89-e055-4140-95de-f1df723db034/c1dd8f61-494c-402f-8e59-08309c64fc3f"
           (reference "U301") (unit 1)
@@
     (pin "1")
     (instances
-      (project "honeycomb-pcb"
+      (project "cluster-pcb"
         (path "/df2b2e89-e055-4140-95de-f1df723db034/c1dd8f61-494c-402f-8e59-08309c64fc3f"
           (reference "#FLG0302") (unit 1)
@@
     (pin "1")
     (instances
-      (project "honeycomb-pcb"
+      (project "cluster-pcb"
         (path "/df2b2e89-e055-4140-95de-f1df723db034/c1dd8f61-494c-402f-8e59-08309c64fc3f"
           (reference "#FLG0304") (unit 1)
@@
     (pin "2")
     (instances
-      (project "honeycomb-pcb"
+      (project "cluster-pcb"
         (path "/df2b2e89-e055-4140-95de-f1df723db034/c1dd8f61-494c-402f-8e59-08309c64fc3f"
           (reference "C302") (unit 1)
@@
     (pin "1")
     (instances
-      (project "honeycomb-pcb"
+      (project "cluster-pcb"
         (path "/df2b2e89-e055-4140-95de-f1df723db034/c1dd8f61-494c-402f-8e59-08309c64fc3f"
           (reference "R301") (unit 1)
@@
     (pin "2")
     (instances
-      (project "honeycomb-pcb"
+      (project "cluster-pcb"
         (path "/df2b2e89-e055-4140-95de-f1df723db034/c1dd8f61-494c-402f-8e59-08309c64fc3f"
           (reference "D301") (unit 1)
@@
     (pin "2")
     (instances
-      (project "honeycomb-pcb"
+      (project "cluster-pcb"
         (path "/df2b2e89-e055-4140-95de-f1df723db034/c1dd8f61-494c-402f-8e59-08309c64fc3f"
           (reference "C301") (unit 1)
@@
     (pin "2")
     (instances
-      (project "honeycomb-pcb"
+      (project "cluster-pcb"
         (path "/df2b2e89-e055-4140-95de-f1df723db034/c1dd8f61-494c-402f-8e59-08309c64fc3f"
           (reference "R302") (unit 1)
@@
     (pin "1")
     (instances
-      (project "honeycomb-pcb"
+      (project "cluster-pcb"
         (path "/df2b2e89-e055-4140-95de-f1df723db034/c1dd8f61-494c-402f-8e59-08309c64fc3f"
           (reference "#FLG0303") (unit 1)
@@
     (pin "1")
     (instances
-      (project "honeycomb-pcb"
+      (project "cluster-pcb"
         (path "/df2b2e89-e055-4140-95de-f1df723db034/c1dd8f61-494c-402f-8e59-08309c64fc3f"
           (reference "C304") (unit 1)
@@
     (pin "1")
     (instances
-      (project "honeycomb-pcb"
+      (project "cluster-pcb"
         (path "/df2b2e89-e055-4140-95de-f1df723db034/c1dd8f61-494c-402f-8e59-08309c64fc3f"
           (reference "M301") (unit 1)
@@
     (pin "2")
     (instances
-      (project "honeycomb-pcb"
+      (project "cluster-pcb"
         (path "/df2b2e89-e055-4140-95de-f1df723db034/c1dd8f61-494c-402f-8e59-08309c64fc3f"
           (reference "Q302") (unit 1)

Commit message: Initial layout
Parts:
- renumbered Q302 to Q301, Q301 to Q302
Changed lines of the file:
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@@
   (symbol (lib_id "Janelia:MOSFET-P-CH-EN_60V_50A") (at 158.75 109.22 0) (unit 1)
     (in_bom yes) (on_board yes) (dnp no) (fields_autoplaced)
-    (property "Reference" "Q301" (at 163.83 109.22 0) (do_not_autoplace)
+    (property "Reference" "Q302" (at 163.83 109.22 0) (do_not_autoplace)
       (effects (font (size 1.27 1.27)) (justify left))
     )
@@
       (project "cluster-pcb"
         (path "/df2b2e89-e055-4140-95de-f1df723db034/c1dd8f61-494c-402f-8e59-08309c64fc3f"
-          (reference "Q301") (unit 1)
+          (reference "Q302") (unit 1)
         )
       )
@@
   (symbol (lib_id "Janelia:MOSFET-N-CH-EN_100V_260mA") (at 113.03 130.81 0) (unit 1)
     (in_bom yes) (on_board yes) (dnp no) (fields_autoplaced)
-    (property "Reference" "Q302" (at 118.11 130.81 0) (do_not_autoplace)
+    (property "Reference" "Q301" (at 118.11 130.81 0) (do_not_autoplace)
       (effects (font (size 1.27 1.27)) (justify left))
     )
@@
       (project "cluster-pcb"
         (path "/df2b2e89-e055-4140-95de-f1df723db034/c1dd8f61-494c-402f-8e59-08309c64fc3f"
-          (reference "Q302") (unit 1)
-        )
-      )
+          (reference "Q301") (unit 1)
+        )
+      )

Commit message: Initial layout
Parts:
- removed M301: Fan_5VDC_25x25x8mm, Janelia:FAN_5VDC_25x25x8mm, symbol Janelia:Fan_5VDC_25x25x8mm
Changed lines of the file:
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@@
   (title_block
     (title "cluster-pcb")
-    (date "2024-07-16")
+    (date "2024-07-17")
     (rev "1.0")
     (company "Howard Hughes Medical Institute")
@@
     (stroke (width 0) (type default))
   )
-  (wire (pts (xy 208.28 127) (xy 208.28 129.54))
-    (stroke (width 0) (type default))
-  )
   (wire (pts (xy 167.64 66.04) (xy 167.64 68.58))
     (stroke (width 0) (type default))
@@
     (stroke (width 0) (type default))
   )
-  (wire (pts (xy 208.28 109.22) (xy 208.28 106.68))
-    (stroke (width 0) (type default))
-  )
   (wire (pts (xy 153.67 109.22) (xy 151.13 109.22))
     (stroke (width 0) (type default))
@@
     (effects (font (size 1.27 1.27)) (justify right bottom))
   )
-  (label "+5V" (at 208.28 106.68 90) (fields_autoplaced)
-    (effects (font (size 1.27 1.27)) (justify left bottom))
-  )
   (label "GND" (at 167.64 68.58 270) (fields_autoplaced)
     (effects (font (size 1.27 1.27)) (justify right bottom))
@@
   (label "+5V" (at 241.3 64.77 0) (fields_autoplaced)
     (effects (font (size 1.27 1.27)) (justify left bottom))
-  )
-  (label "GND" (at 208.28 129.54 270) (fields_autoplaced)
-    (effects (font (size 1.27 1.27)) (justify right bottom))
   )
   (label "GND" (at 151.13 68.58 270) (fields_autoplaced)
@@
         )
       )
-    )
-  )
-  (symbol (lib_id "Janelia:Fan_5VDC_25x25x8mm") (at 208.28 118.11 0) (unit 1)
-    (in_bom no) (on_board yes) (dnp no) (fields_autoplaced)
-    (property "Reference" "M301" (at 212.09 118.11 0) (do_not_autoplace)
-      (effects (font (size 1.27 1.27)) (justify left))
-    )
-    (property "Value" "Fan_5VDC_25x25x8mm" (at 208.28 113.03 0) (do_not_autoplace)
-      (effects (font (size 1.27 1.27)) (justify top) hide)
-    )
-    (property "Footprint" "Janelia:FAN_5VDC_25x25x8mm" (at 208.28 100.33 0)
-      (effects (font (size 1.27 1.27)) hide)
-    )
-    (property "Datasheet" "~" (at 208.28 101.6 0)
-      (effects (font (size 1.27 1.27)) hide)
-    )
-    (property "Synopsis" "FAN AXIAL 25X8MM 5VDC WIRE" (at 208.28 111.76 0)
-      (effects (font (size 1.27 1.27)) hide)
-    )
-    (property "Manufacturer" "ebm-papst Inc." (at 208.28 109.22 0)
-      (effects (font (size 1.27 1.27)) hide)
-    )
-    (property "Manufacturer Part Number" "255M" (at 208.28 110.49 0) (do_not_autoplace)
-      (effects (font (size 1.27 1.27)) hide)
-    )
-    (property "Vendor" "Digi-Key" (at 208.28 106.68 0)
-      (effects (font (size 1.27 1.27)) hide)
-    )
-    (property "Vendor Part Number" "381-2353-ND" (at 208.28 104.14 0)
-      (effects (font (size 1.27 1.27)) hide)
-    )
-    (property "LCSC" "" (at 208.28 118.11 0)
-      (effects (font (size 1.27 1.27)) hide)
-    )
-    (property "Sim.Enable" "0" (at 208.28 118.11 0)
-      (effects (font (size 1.27 1.27)) hide)
-    )
-    (pin "2")
-    (pin "3")
-    (pin "1")
-    (instances
-      (project "cluster-pcb"
-        (path "/df2b2e89-e055-4140-95de-f1df723db034/c1dd8f61-494c-402f-8e59-08309c64fc3f"
-          (reference "M301") (unit 1)
-        )
-      )
