File: cluster-pcb/power.kicad_sch (KiCad schematic)
At the start: 10 parts, among them T301 TERM_BLK_HDR_2POS_90DEG_0.2IN, U301 TPSM365R6V5RDNR

Commit message: Finished v2.1
Parts:
- C305: LCSC C2182652 -> C6119904; Manufacturer TDK Corporation -> HRE; Manufacturer Part Number C2012X5R1A476M125AC -> CGA0805X5R476M100MT; Vendor Digi-Key -> JLCPCB; Vendor Part Number 445-8239-1-ND -> C6119904
Changed lines of the file:
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@@
   (title_block
     (title "cluster-pcb")
-    (date "2024-10-21")
+    (date "2024-10-22")
     (rev "2.1")
     (company "Howard Hughes Medical Institute")
@@
       (effects (font (size 1.524 1.524)))
     )
-    (property "Vendor" "Digi-Key" (at 208.28 116.84 0)
-      (effects (font (size 1.524 1.524)) hide)
-    )
-    (property "Vendor Part Number" "445-8239-1-ND" (at 210.82 114.3 0)
+    (property "Vendor" "JLCPCB" (at 208.28 116.84 0)
+      (effects (font (size 1.524 1.524)) hide)
+    )
+    (property "Vendor Part Number" "C6119904" (at 210.82 114.3 0)
       (effects (font (size 1.524 1.524)) hide)
     )
@@
       (effects (font (size 1.27 1.27)) hide)
     )
-    (property "Manufacturer" "TDK Corporation" (at 205.74 121.92 0)
-      (effects (font (size 1.27 1.27)) hide)
-    )
-    (property "Manufacturer Part Number" "C2012X5R1A476M125AC" (at 205.74 121.92 0)
+    (property "Manufacturer" "HRE" (at 205.74 121.92 0)
+      (effects (font (size 1.27 1.27)) hide)
+    )
+    (property "Manufacturer Part Number" "CGA0805X5R476M100MT" (at 205.74 121.92 0)
       (effects (font (size 1.27 1.27)) hide)
     )
@@
       (effects (font (size 1.524 1.524)) hide)
     )
-    (property "LCSC" "C2182652" (at 205.74 121.92 0)
-      (effects (font (size 1.27 1.27)) hide)
-    )
+    (property "LCSC" "C6119904" (at 205.74 121.92 0)
+      (effects (font (size 1.27 1.27)) hide)
+    )
