File: cluster-pcb/multiplexer.kicad_sch (KiCad schematic)
At the start: 3 parts, among them U1301 MUX507

Commit message: Routed most tracks
Parts:
- removed C1301: 0.1uF_100V, Janelia:C_0402_1005Metric, symbol Janelia:C_0.1uF_100V_0402
- added C1301: 1uF_35V, Janelia:C_0402_1005Metric, symbol Janelia:C_1uF_35V_0402
Connections:
- net GND: now also C1301.2
- net VAA: now also C1301.1
Changed lines of the file:
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@@
     (effects (font (size 1.27 1.27)) (justify left))
+  )
+  (symbol (lib_id "Janelia:C_1uF_35V_0402") (at 114.3 43.18 0) (unit 1)
+    (in_bom yes) (on_board yes) (dnp no)
+    (property "Reference" "C1301" (at 116.84 41.91 0)
+      (effects (font (size 1.016 1.016)) (justify left))
+    )
+    (property "Value" "1uF_35V" (at 116.84 44.45 0)
+      (effects (font (size 0.762 0.762)) (justify left))
+    )
+    (property "Footprint" "Janelia:C_0402_1005Metric" (at 115.2652 46.99 0)
+      (effects (font (size 0.762 0.762)) hide)
+    )
+    (property "Datasheet" "" (at 114.3 43.18 0)
+      (effects (font (size 1.524 1.524)) hide)
+    )
+    (property "Vendor" "Digi-Key" (at 116.84 38.1 0)
+      (effects (font (size 1.524 1.524)) hide)
+    )
+    (property "Vendor Part Number" "1276-6796-1-ND" (at 119.38 35.56 0)
+      (effects (font (size 1.524 1.524)) hide)
+    )
+    (property "Synopsis" "CAP CER 1UF 35V X5R" (at 121.92 33.02 0)
+      (effects (font (size 1.524 1.524)) hide)
+    )
+    (property "Package" "0402" (at 114.3 43.18 0)
+      (effects (font (size 1.27 1.27)) hide)
+    )
+    (property "Manufacturer" "Samsung Electro-Mechanics" (at 114.3 43.18 0)
+      (effects (font (size 1.27 1.27)) hide)
+    )
+    (property "Manufacturer Part Number" "CL05A105KL5NRNC" (at 114.3 43.18 0)
+      (effects (font (size 1.27 1.27)) hide)
+    )
+    (property "LCSC" "C307413" (at 114.3 43.18 0)
+      (effects (font (size 1.27 1.27)) hide)
+    )
+    (pin "2")
+    (pin "1")
+    (instances
+      (project "cluster-pcb"
+        (path "/df2b2e89-e055-4140-95de-f1df723db034/6263f048-a0b9-4a20-a0ec-2762a3a0da32"
+          (reference "C1301") (unit 1)
+        )
+      )
+    )
   )
   (symbol (lib_id "Janelia:Multiplexer_2chan_8to1_MUX507IDWR") (at 124.46 90.17 0) (unit 1)
@@
         )
       )
-    )
-  )
-  (symbol (lib_id "Janelia:C_0.1uF_100V_0402") (at 114.3 43.18 0) (unit 1)
-    (in_bom yes) (on_board yes) (dnp no)
-    (property "Reference" "C1301" (at 116.84 41.91 0)
-      (effects (font (size 1.016 1.016)) (justify left))
-    )
-    (property "Value" "0.1uF_100V" (at 116.84 44.45 0)
-      (effects (font (size 0.762 0.762)) (justify left))
-    )
-    (property "Footprint" "Janelia:C_0402_1005Metric" (at 115.2652 46.99 0)
-      (effects (font (size 0.762 0.762)) hide)
-    )
-    (property "Datasheet" "" (at 114.3 40.64 0)
-      (effects (font (size 1.524 1.524)) hide)
-    )
-    (property "Vendor" "Digi-Key" (at 116.84 38.1 0)
-      (effects (font (size 1.524 1.524)) hide)
-    )
-    (property "Vendor Part Number" "490-10458-1-ND" (at 119.38 35.56 0)
-      (effects (font (size 1.524 1.524)) hide)
-    )
-    (property "Synopsis" "CAP CER 0.1UF 100V X5R" (at 121.92 33.02 0)
-      (effects (font (size 1.524 1.524)) hide)
-    )
-    (property "Manufacturer" "Murata Electronics" (at 114.3 43.18 0)
-      (effects (font (size 1.27 1.27)) hide)
-    )
-    (property "Manufacturer Part Number" "GRM155R62A104KE14D" (at 114.3 43.18 0)
-      (effects (font (size 1.27 1.27)) hide)
-    )
-    (property "Package" "0402" (at 114.3 43.18 0)
-      (effects (font (size 1.27 1.27)) hide)
-    )
-    (property "LCSC" "C162178" (at 114.3 43.18 0)
-      (effects (font (size 1.27 1.27)) hide)
-    )
-    (pin "1")
-    (pin "2")
-    (instances
-      (project "cluster-pcb"
-        (path "/df2b2e89-e055-4140-95de-f1df723db034/6263f048-a0b9-4a20-a0ec-2762a3a0da32"
-          (reference "C1301") (unit 1)
-        )
-      )

Commit message: Update metadata
Parts:
- U1301: footprint DW28_TEX -> Janelia:DW28_TEX; LCSC (none) -> C193367; Manufacturer (none) -> Texas Instruments; Manufacturer Part Number (none) -> MUX507IDWR; Package (none) -> SOIC-28-300mil; Synopsis (none) -> IC MUX DUAL 8:1 200OHM; Vendor (none) -> Digi-Key; Vendor Part Number (none) -> 296-47545-1-ND
Changed lines of the file:
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@@
       (effects (font (size 1.524 1.524)))
     )
-    (property "Footprint" "DW28_TEX" (at 124.46 33.02 0)
+    (property "Footprint" "Janelia:DW28_TEX" (at 124.46 33.02 0)
       (effects (font (size 1.27 1.27) italic) hide)
     )
-    (property "Datasheet" "MUX507IDWR" (at 124.46 30.48 0)
+    (property "Datasheet" "" (at 124.46 30.48 0)
       (effects (font (size 1.27 1.27) italic) hide)
     )
+    (property "Synopsis" "IC MUX DUAL 8:1 200OHM" (at 124.46 90.17 0)
+      (effects (font (size 1.27 1.27)) hide)
+    )
+    (property "Package" "SOIC-28-300mil" (at 124.46 90.17 0)
+      (effects (font (size 1.27 1.27)) hide)
+    )
+    (property "Manufacturer" "Texas Instruments" (at 124.46 90.17 0)
+      (effects (font (size 1.27 1.27)) hide)
+    )
+    (property "Manufacturer Part Number" "MUX507IDWR" (at 124.46 90.17 0)
+      (effects (font (size 1.27 1.27)) hide)
+    )
+    (property "Vendor" "Digi-Key" (at 124.46 90.17 0)
+      (effects (font (size 1.27 1.27)) hide)
+    )
+    (property "Vendor Part Number" "296-47545-1-ND" (at 124.46 90.17 0)
+      (effects (font (size 1.27 1.27)) hide)
+    )
+    (property "LCSC" "C193367" (at 124.46 90.17 0)
+      (effects (font (size 1.27 1.27)) hide)
+    )
     (pin "9")
