File: cluster-pcb/audio.kicad_sch (KiCad schematic)
At the start: 8 parts, among them U1401 TPA6204A1DRBR

Commit message: Fix ERC issues
Other:
- company: (none) -> Howard Hughes Medical Institute
- title: (none) -> cluster-pcb
Changed lines of the file:
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@@
 (kicad_sch (version 20230121) (generator eeschema)
   (paper "A4")
+  (title_block
+    (title "cluster-pcb")
+    (date "2024-09-13")
+    (rev "1.2")
+    (company "Howard Hughes Medical Institute")
+  )
   (wire (pts (xy 129.54 116.84) (xy 129.54 119.38))
     (stroke (width 0) (type default))
